Commit message: update robot model

File: sf_robot/config/sf1-1.xacro (robot description, xacro)
@@ -5,8 +5,203 @@
 	xmlns:interface="http://playerstage.sourceforge.net/gazebo/xmlschema/#interface"
 	xmlns:xacro="http://ros.org/wiki/xacro">
-    <include filename="$(find p2os_urdf)/defs/pioneer3dx.xacro"/>
-    <include filename="$(find pr2_description)/urdf/sensors/hokuyo_lx30_laser.urdf.xacro" />
-    <xacro:hokuyo_lx30_laser_v0 name="base_laser_front" parent="base" ros_topic="scan_front" update_rate="20" min_angle="-2.2689" max_angle="2.2689" >
-      <origin xyz="0.13 0.0 0.045" rpy="0 0 0" />
-    </xacro:hokuyo_lx30_laser_v0>
+	<!-- Base -->
+	<include filename="$(find p2os_urdf)/defs/pioneer3dx.xacro" />
+	<include filename="$(find sf_robot)/config/hokuyo_laser.xacro" />
+	<xacro:hokuyo_04lx_laser_ug01 name="base_laser_front"
+		parent="base" ros_topic="scan_front" update_rate="10" min_angle="-2.094"
+		max_angle="2.094">
+		<origin rpy="0 0 0" xyz="0.15 0.0 0.245" />
+	</xacro:hokuyo_04lx_laser_ug01>
+	<joint name="base_plate_joint" type="fixed">
+		<origin rpy="0 0 0" xyz="0 0 0.0085" />
+		<parent link="top_plate" />
+		<child link="base_plate_link" />
+	</joint>
+	<link name="base_plate_link">
+		<visual>
+			<inertial>
+				<mass value="0.1" />
+				<origin xyz="0 0 0" />
+				<inertia ixx="1" ixy="0" ixz="0" iyy="1" iyz="0" izz="1" />
+			</inertial>
+			<origin rpy="0 0 0" xyz="0 0 0" />
+			<geometry name="top_geom">
+				<mesh filename="package://p2os_urdf/meshes/p3dx_meshes/top.stl" />
+			</geometry>
+			<material name="wood">
+				<color rgba="0.96 0.86 0.57 1.0" />
+			</material>
+		</visual>
+	</link>
+	<!-- Tray -->
+	<xacro:macro name="tray" params="name parent *origin">
+		<joint name="${name}_joint" type="fixed">
+			<insert_block name="origin" />
+			<parent link="${parent}_link" />
+			<child link="${name}_link" />
+		</joint>
+		<link name="${name}_link">
+			<inertial>
+				<mass value="2" />
+				<origin xyz="0 0 0" rpy="0 0 0" />
+				<inertia ixx="0.001" ixy="0.0" ixz="0.0" iyy="0.001" iyz="0.0"
+					izz="0.001" />
+			</inertial>
+			<visual>
+				<origin xyz="0 0 0" rpy="0 0 0" />
+				<geometry>
+					<box size="0.23 0.325 0.18" />
+				</geometry>
+				<material name="wood">
+					<color rgba="0.96 0.86 0.57 1.0" />
+				</material>
+			</visual>
+			<collision>
+				<origin xyz="0 0 0" rpy="0 0 0" />
+				<geometry>
+					<box size="0.23 0.325 0.18" />
+				</geometry>
+			</collision>
+		</link>
+	</xacro:macro>
+	<xacro:tray name="tray" parent="base">
+		<origin rpy="0 0 0" xyz="0.01 0 0.645" />
+	</xacro:tray>
+	<!-- Head -->
+	<xacro:macro name="camera" params="name parent *origin">
+		<joint name="${name}_joint" type="fixed">
+			<insert_block name="origin" />
+			<parent link="${parent}_link" />
+			<child link="${name}_link" />
+		</joint>
+		<link name="${name}_link">
+			<inertial>
+				<mass value="0.01" />
+				<origin xyz="0 0 0" rpy="0 0 0" />
+				<inertia ixx="0.001" ixy="0.0" ixz="0.0" iyy="0.001" iyz="0.0"
+					izz="0.001" />
+			</inertial>
+			<visual>
+				<origin xyz="0 0 0" rpy="0 0 0" />
+				<geometry>
+					<cylinder length="0.002" radius="0.015" />
+				</geometry>
+				<material name="black">
+					<color rgba="0.07 0.07 0.07 1.0" />
+				</material>
+			</visual>
+			<collision>
+				<origin xyz="0 0 0" rpy="0 0 0" />
+				<geometry>
+					<cylinder length="0.002" radius="0.015" />
+				</geometry>
+			</collision>
+		</link>
+	</xacro:macro>
+	<xacro:macro name="eye" params="name parent *origin">
+		<joint name="${name}_joint" type="fixed">
+			<insert_block name="origin" />
+			<parent link="${parent}_link" />
+			<child link="${name}_link" />
+		</joint>
+		<link name="${name}_link">
+			<inertial>
+				<mass value="0.01" />
+				<origin xyz="0 0 0" rpy="0 0 0" />
+				<inertia ixx="0.001" ixy="0.0" ixz="0.0" iyy="0.001" iyz="0.0"
+					izz="0.001" />
+			</inertial>
+			<visual>
+				<origin xyz="0 0 0" rpy="0 0 0" />
+				<geometry>
+					<cylinder length="0.015" radius="0.03" />
+				</geometry>
+				<material name="white">
+					<color rgba="0.98 0.98 0.90 1.0" />
+				</material>
+			</visual>
+			<collision>
+				<origin xyz="0 0 0" rpy="0 0 0" />
+				<geometry>
+					<cylinder length="0.015" radius="0.03" />
+				</geometry>
+			</collision>
+		</link>
+	</xacro:macro>
+	<xacro:macro name="head" params="name parent *origin">
+		<joint name="${name}_joint" type="fixed">
+			<insert_block name="origin" />
+			<parent link="${parent}_link" />
+			<child link="${name}_link" />
+		</joint>
+		<link name="${name}_link">
+			<inertial>
+				<mass value="0.1" />
+				<origin xyz="0 0 -0.05" rpy="0 0 0" />
+				<inertia ixx="0.001" ixy="0.0" ixz="0.0" iyy="0.001" iyz="0.0"
+					izz="0.001" />
+			</inertial>
+			<visual>
+				<origin xyz="0 0 -0.05" rpy="0 0 0" />
+				<geometry>
+					<cylinder length="0.10" radius="0.11" />
+				</geometry>
+				<material name="grey">
+					<color rgba="0.5 0.5 0.5 1.0" />
+				</material>
+			</visual>
+			<collision>
+				<origin xyz="0 0 -0.05" rpy="0 0 0" />
+				<geometry>
+					<cylinder length="0.10" radius="0.11" />
+				</geometry>
+			</collision>
+		</link>
+		<xacro:eye name="eye_r" parent="${name}">
+			<origin rpy="0.23 1.57 0" xyz="0.12 -0.06 -0.05" />
+		</xacro:eye>
+		<xacro:eye name="eye_l" parent="${name}">
+			<origin rpy="-0.23 1.57 0" xyz="0.12 0.06 -0.05" />
+		</xacro:eye>
+		<xacro:camera name="camera" parent="${name}">
+			<origin rpy="0 1.57 0" xyz="0.11 0.00 -0.07" />
+		</xacro:camera>
+	</xacro:macro>
+	<xacro:head name="head" parent="base">
+		<origin rpy="0 0 0" xyz="0 0 1.045" />
+	</xacro:head>
+	<!--Body -->
+	<xacro:macro name="body" params="name parent *origin">
+		<joint name="${name}_joint" type="fixed">
+			<insert_block name="origin" />
+			<parent link="${parent}_link" />
+			<child link="${name}_link" />
+		</joint>
+		<link name="${name}_link">
+			<inertial>
+				<mass value="10" />
+				<origin xyz="0 0 0.2525" rpy="0 0 0" />
+				<inertia ixx="0.001" ixy="0.0" ixz="0.0" iyy="0.001" iyz="0.0"
+					izz="0.001" />
+			</inertial>
+			<visual>
+				<origin xyz="0 0 0.2525" rpy="0 0 0" />
+				<geometry>
+					<box size="0.30 0.33 0.505" />
+				</geometry>
+				<material name="white">
+					<color rgba="0.98 0.98 0.90 1.0" />
+				</material>
+			</visual>
+			<collision>
+				<origin xyz="0 0 0.2525" rpy="0 0 0" />
+				<geometry>
+					<box size="0.30 0.33 0.505" />
+				</geometry>
+			</collision>
+		</link>
+	</xacro:macro>
+	<xacro:body name="body" parent="base">
+		<origin rpy="0 0 0" xyz="-0.04 0 0.245" />
+	</xacro:body>
 </robot>

Commit message: Patch 'continuous' joints for rviz

File: sf_robot/config/sf1-1.xacro (robot description, xacro)
@@ -34,4 +34,15 @@
 		</visual>
 	</link>
+    <!-- Override the 'continuous' joint from p3dx.xacro -->
+    <joint name="base_swivel_joint_fixed" type="fixed">
+        <origin xyz="-0.185 0 0.055" rpy="0 0 0"/>
+        <parent link="base_link"/>
+        <child link="swivel"/>
+    </joint>
+    <joint name="swivel_hubcap_joint_fixed" type="fixed">
+        <origin xyz="-0.026 0 -0.016" rpy="0 0 0"/>
+        <parent link="swivel"/>
+        <child link="center_wheel"/>
+    </joint>
 	<!-- Tray -->
 	<xacro:macro name="tray" params="name parent *origin">

Commit message: Finish updates for WB7, add neck to Rviz model (visually broken, but functional)

File: sf_robot/config/sf1-1.xacro (robot description, xacro)
@@ -79,4 +79,56 @@
 		<origin rpy="0 0 0" xyz="0.01 0 0.645" />
 	</xacro:tray>
+    <!-- Neck -->
+    <include filename="$(find sf_dynamixel)/defs/dynamixel_ax12.xacro" />
+    <include filename="$(find sf_dynamixel)/defs/fp04_02.xacro" />
+    <xacro:macro name="neck" params="name parent *origin">
+        <xacro:ax12
+                name="neck_lower"
+                parent="${parent}"
+                minPosition="-1.5705"
+                maxPosition="1.5707"
+                maxVelocity="1">
+            <insert_block name="origin"/>
+        </xacro:ax12>
+        <xacro:fp04_02
+                name="neck_lower_hinge"
+                parent="neck_lower">
+        </xacro:fp04_02>
+        <xacro:ax12
+                name="neck_upper"
+                parent="neck_lower_hinge"
+                minPosition="-1.5705"
+                maxPosition="1.5707"
+                maxVelocity="1">
+            <origin rpy="1.5707 0 1.5707" xyz="0 -0.0635 0"/>
+        </xacro:ax12>
+        <xacro:fp04_02
+                name="neck_upper_hinge"
+                parent="neck_upper">
+        </xacro:fp04_02>
+        <xacro:ax12
+                name="head_tilt"
+                parent="neck_upper_hinge"
+                minPosition="-1.5705"
+                maxPosition="1.5707"
+                maxVelocity="1">
+            <origin rpy="0 0 1.5707" xyz="0 -0.0635 0"/>
+        </xacro:ax12>
+        <xacro:fp04_02
+                name="head_tilt_hinge"
+                parent="head_tilt">
+        </xacro:fp04_02>
+        <xacro:ax12inverted
+                name="head_pan"
+                parent="head_tilt_hinge"
+                minPosition="-1.5705"
+                maxPosition="1.5707"
+                maxVelocity="1">
+            <origin rpy="0 0 1.5707" xyz="0 -0.0635 0"/>
+        </xacro:ax12inverted>
+    </xacro:macro>
+    <xacro:neck name="neck" parent="base">
+        <origin rpy="0 1.5707 0" xyz="0 0 0.79" />
+    </xacro:neck>
 	<!-- Head -->
 	<xacro:macro name="camera" params="name parent *origin">
@@ -179,6 +231,6 @@
 		</xacro:camera>
 	</xacro:macro>
-	<xacro:head name="head" parent="base">
-		<origin rpy="0 0 0" xyz="0 0 1.045" />
+	<xacro:head name="head" parent="head_pan">
+		<origin rpy="0 1.5707 3.14159" xyz="-0.05 0 0" />
 	</xacro:head>
 	<!--Body -->

Commit message: Update sf1-1.xacro
Change tray from fixed to 'prismatic' joint

File: sf_robot/config/sf1-1.xacro (robot description, xacro)
@@ -47,8 +47,9 @@
 	<!-- Tray -->
 	<xacro:macro name="tray" params="name parent *origin">
-		<joint name="${name}_joint" type="fixed">
-			<insert_block name="origin" />
-			<parent link="${parent}_link" />
-			<child link="${name}_link" />
+		<joint name="${name}_joint" type="prismatic">
+			<insert_block name="origin" />
+			<parent link="${parent}_link" />
+			<child link="${name}_link" />
+			<limit lower="0.0" upper="0.1" velocity="0.5"/>
 		</joint>
 		<link name="${name}_link">

Commit message: Update sf1-1.xacro
Add axis to tray joint

File: sf_robot/config/sf1-1.xacro (robot description, xacro)
@@ -52,4 +52,5 @@
 			<child link="${name}_link" />
 			<limit lower="0.0" upper="0.1" velocity="0.5"/>
+			<axis xyz="1 0 0"/>
 		</joint>
 		<link name="${name}_link">

Commit message: correct sunflower tray joint range

File: sf_robot/config/sf1-1.xacro (robot description, xacro)
@@ -51,5 +51,5 @@
 			<parent link="${parent}_link" />
 			<child link="${name}_link" />
-			<limit lower="0.0" upper="0.1" velocity="0.5"/>
+			<limit effort="0" lower="0.0" upper="0.15" velocity="0.5"/>
 			<axis xyz="1 0 0"/>
 		</joint>

Commit message: fix head pan in webots, head_tilt in rviz

File: sf_robot/config/sf1-1.xacro (robot description, xacro)
@@ -117,5 +117,5 @@
 		<xacro:ax12inverted name="head_pan" parent="neck_upper_hinge"
 			minPosition="-1.5707" maxPosition="1.5707" maxVelocity="1">
-			<origin rpy="0 0 0" xyz="0 0 0" />
+			<origin rpy="0 0 -1.57079" xyz="0 0 0" />
 		</xacro:ax12inverted>
 		<xacro:ax12 name="head_tilt" parent="head_pan" minPosition="-1.5707"
@@ -272,5 +272,5 @@
 	</xacro:macro>
 	<xacro:head name="head" parent="head_tilt_hinge">
-		<origin rpy="0 0 -1.5707" xyz="0 0 0" />
+		<origin rpy="0 0 0" xyz="0 0 0" />
 	</xacro:head>
 	<!--Body -->
