Commit message: fix laser frame_ids in urdf, more detailed person urdf

File: person_sim/config/hokuyo_laser.xacro (robot description, xacro)
@@ -34,7 +34,7 @@
 			<origin xyz="0 0 0.041" rpy="0 0 0" />
 			<parent link="${name}_link" />
-			<child link="${name}_scan_link" />
+			<child link="${ros_topic}" />
 		</joint>
-		<link name="${name}_scan_link" type="laser">
+		<link name="${ros_topic}" type="laser">
 			<inertial>
 				<mass value="0.01" />

File: person_sim/config/person.xacro (robot description, xacro)
@@ -6,20 +6,214 @@
 	xmlns:xacro="http://ros.org/wiki/xacro">
 	<link name="base_link">
-		<visual>
-			<geometry>
-				<cylinder length="2.0" radius="0.18" />
-			</geometry>
-		</visual>
 	</link>
+	<xacro:macro name="torso" params="name parent *origin">
+		<joint name="${name}_joint" type="fixed">
+			<insert_block name="origin" />
+			<parent link="${parent}_link" />
+			<child link="${name}_link" />
+		</joint>
+		<link name="${name}_link">
+			<visual>
+				<origin xyz="0 0 0.3" rpy="0 0 0" />
+				<geometry>
+					<box size="0.2 0.3 0.6" />
+				</geometry>
+				<material name="shirt">
+					<color rgba="0.611765 0.0156863 0.0156863 1.0" />
+				</material>
+			</visual>
+			<collision>
+				<origin xyz="0 0 0.3" rpy="0 0 0" />
+				<geometry>
+					<box size="0.2 0.3 0.6" />
+				</geometry>
+			</collision>
+		</link>
+		<joint name="${name}_shoulders_joint" type="fixed">
+			<origin xyz="0 0 0.6" rpy="0 0 1.57079" />
+			<parent link="${name}_link" />
+			<child link="${name}_shoulders_link" />
+		</joint>
+		<link name="${name}_shoulders_link">
+			<visual>
+				<origin xyz="0 0 0" rpy="0 1.57079 0" />
+				<geometry>
+					<cylinder length="0.6" radius="0.1" />
+				</geometry>
+				<material name="shirt">
+					<color rgba="0.611765 0.0156863 0.0156863 1.0" />
+				</material>
+			</visual>
+			<collision>
+				<origin xyz="0 0 0" rpy="0 1.57079 0" />
+				<geometry>
+					<cylinder length="0.6" radius="0.1" />
+				</geometry>
+			</collision>
+		</link>
+		<gazebo reference="${name}_link">
+			<material>Gazebo/Red</material>
+		</gazebo>
+		<xacro:arm name="${name}_arm_right" parent="${name}_shoulders">
+			<origin rpy="0 0 0" xyz="0.23 0 -0.05" />
+		</xacro:arm>
+		<xacro:arm name="${name}_arm_left" parent="${name}_shoulders">
+			<origin rpy="0 0 0" xyz="-0.23 0 -0.05" />
+		</xacro:arm>
+		<xacro:head name="${name}_head" parent="${name}_shoulders">
+			<origin rpy="0 0 0" xyz="0 0 0.07" />
+		</xacro:head>
+	</xacro:macro>
+	<xacro:macro name="head" params="name parent *origin">
+		<joint name="${name}_bottom_joint" type="fixed">
+			<insert_block name="origin" />
+			<parent link="${parent}_link" />
+			<child link="${name}_link" />
+		</joint>
+		<link name="${name}_link">
+		</link>
+		<joint name="${name}_joint" type="fixed">
+			<origin xyz="0 0 0.08" rpy="0 0 0" />
+			<parent link="${name}_link" />
+			<child link="${name}_bottom_link" />
+		</joint>
+		<link name="${name}_bottom_link">
+			<visual>
+				<geometry>
+					<sphere radius="0.08" />
+				</geometry>
+				<material name="skin">
+					<color rgba="1 0.803922 0.552941 1.0" />
+				</material>
+			</visual>
+			<collision>
+				<geometry>
+					<sphere radius="0.08" />
+				</geometry>
+			</collision>
+		</link>
+		<joint name="${name}_middle_joint" type="fixed">
+			<origin xyz="0 0 0.035" rpy="0 0 0" />
+			<parent link="${name}_bottom_link" />
+			<child link="${name}_middle_link" />
+		</joint>
+		<link name="${name}_middle_link">
+			<visual>
+				<geometry>
+					<cylinder length="0.07" radius="0.08" />
+				</geometry>
+				<material name="skin">
+					<color rgba="1 0.803922 0.552941 1.0" />
+				</material>
+			</visual>
+			<collision>
+				<geometry>
+					<cylinder length="0.07" radius="0.08" />
+				</geometry>
+			</collision>
+		</link>
+		<joint name="${name}_top_joint" type="fixed">
+			<origin xyz="0 0 0.15" rpy="0 0 0" />
+			<parent link="${name}_link" />
+			<child link="${name}_top_link" />
+		</joint>
+		<link name="${name}_top_link">
+			<visual>
+				<geometry>
+					<sphere radius="0.08" />
+				</geometry>
+				<material name="skin">
+					<color rgba="1 0.803922 0.552941 1.0" />
+				</material>
+			</visual>
+			<collision>
+				<geometry>
+					<sphere radius="0.08" />
+				</geometry>
+			</collision>
+		</link>
+		<gazebo reference="${name}_bottom_link">
+			<material>Gazebo/Grey</material>
+		</gazebo>
+		<gazebo reference="${name}_middle_link">
+			<material>Gazebo/SmileyHappy</material>
+		</gazebo>
+		<gazebo reference="${name}_top_link">
+			<material>Gazebo/Grey</material>
+		</gazebo>
+	</xacro:macro>
+	<xacro:macro name="arm" params="name parent *origin">
+		<joint name="${name}_joint" type="fixed">
+			<insert_block name="origin" />
+			<parent link="${parent}_link" />
+			<child link="${name}_link" />
+		</joint>
+		<link name="${name}_link">
+			<visual>
+				<origin xyz="0 0 -0.225" rpy="0 0 0" />
+				<geometry>
+					<cylinder length="0.45" radius="0.07" />
+				</geometry>
+				<material name="skin">
+					<color rgba="1 0.803922 0.552941 1.0" />
+				</material>
+			</visual>
+			<collision>
+				<origin xyz="0 0 -0.225" rpy="0 0 0" />
+				<geometry>
+					<cylinder length="0.45" radius="0.07" />
+				</geometry>
+			</collision>
+		</link>
+		<gazebo reference="${name}_link">
+			<material>Gazebo/Grey</material>
+		</gazebo>
+	</xacro:macro>
+	<xacro:macro name="leg" params="name parent *origin">
+		<joint name="${name}_joint" type="fixed">
+			<insert_block name="origin" />
+			<parent link="${parent}_link" />
+			<child link="${name}_link" />
+		</joint>
+		<link name="${name}_link">
+			<visual>
+				<origin xyz="0 0 0.375" rpy="0 0 0" />
+				<geometry>
+					<cylinder length="0.65" radius="0.07" />
+				</geometry>
+				<material name="blue">
+					<color rgba="0.14902 0.294118 0.560784 1.0" />
+				</material>
+			</visual>
+			<collision>
+				<origin xyz="0 0 0.375" rpy="0 0 0" />
+				<geometry>
+					<cylinder length="0.65" radius="0.07" />
+				</geometry>
+			</collision>
+		</link>
+		<gazebo reference="${name}_link">
+			<material>Gazebo/Blue</material>
+		</gazebo>
+	</xacro:macro>
 	<include filename="$(find person_sim)/config/hokuyo_laser.xacro" />
 	<xacro:hokuyo_04lx_laser_ug01 name="base_laser_front"
 		parent="base" ros_topic="scan_front" update_rate="10" min_angle="-2.094"
 		max_angle="2.094">
-		<origin rpy="0 0 0" xyz="0.15 0.0 0.245" />
+		<origin rpy="0 0 0" xyz="0.10 0.0 0.05" />
 	</xacro:hokuyo_04lx_laser_ug01>
 	<xacro:hokuyo_04lx_laser_ug01 name="base_laser_back"
-		parent="base" ros_topic="scan_front" update_rate="10" min_angle="-2.094"
+		parent="base" ros_topic="scan_back" update_rate="10" min_angle="-2.094"
 		max_angle="2.094">
-		<origin rpy="0 0 3.14159" xyz="-0.15 0.0 0.245" />
+		<origin rpy="0 0 3.14159" xyz="-0.10 0.0 0.05" />
 	</xacro:hokuyo_04lx_laser_ug01>
+	<xacro:torso name="torso" parent="base">
+		<origin rpy="0 0 0" xyz="0 0 0.65" />
+	</xacro:torso>
+	<xacro:leg name="leg_right" parent="base">
+		<origin rpy="0 0 0" xyz="0 -0.1 0" />
+	</xacro:leg>
+	<xacro:leg name="leg_left" parent="base">
+		<origin rpy="0 0 0" xyz="0 0.1 0" />
+	</xacro:leg>
 </robot>
