Commit message: begin corrections for broken dynamixel joints

File: sf_dynamixel/defs/dynamixel_ax12.xacro (robot description, xacro)
@@ -4,5 +4,34 @@
     xmlns:interface="http://playerstage.sourceforge.net/gazebo/xmlschema/#interface"
     xmlns:sensor="http://playerstage.sourceforge.net/gazebo/xmlschema/#sensor" xmlns:xacro="http://ros.org/wiki/xacro">
-    <xacro:macro name="ax12" params="name parent minPosition maxPosition maxVelocity *origin">
+    <xacro:macro name="ax12" params="name parent minPosition maxPosition maxVelocity">
+        <joint name="${name}_joint" type="revolute">
+            <parent link="${parent}_link"/>
+            <child link="${name}_link"/>
+            <origin xyz="0.0385 0 0" rpy="1.5707 0 0"/>
+            <axis xyz="0 0 1"/>
+            <limit effort="0" lower="${minPosition}"
+                upper="${maxPosition}" velocity="${maxVelocity}"/>
+        </joint>
+        <link name="${name}_link">
+            <collision>
+                <geometry>
+                    <box size="0.050 0.038 0.032"/>
+                </geometry>
+                <origin rpy="-1.5707 0 0" xyz="-0.0385 0 0"/>
+            </collision>
+            <visual>
+                <geometry name="ax12mesh">
+                    <mesh
+                        filename="package://sf_dynamixel/meshes/ax12_box_plain.stl" scale="0.001 0.001 0.001"/>
+                </geometry>
+                <!-- xyz 0.050 0.038 0.032 -->
+                <origin rpy="0 0 0" xyz="0.0135 0 0"/>
+                <material name="black_plastic">
+                    <color rgba="0.3 0.3 0.3 1"/>
+                </material>
+            </visual>
+        </link>
+    </xacro:macro>
+    <xacro:macro name="ax12old" params="name parent minPosition maxPosition maxVelocity *origin">
         <joint name="${name}_joint" type="revolute">
             <parent link="${parent}_link"/>
@@ -23,6 +52,5 @@
                 <geometry name="ax12mesh">
                     <mesh
-                        filename="package://sf_dynamixel/defs/ax12_box_plain.stl"
-                        scale="0.001 0.001 0.001"/>
+                        filename="package://sf_dynamixel/meshes/ax12_box_plain.stl" scale="0.001 0.001 0.001"/>
                 </geometry>
                 <!-- xyz 0.050 0.038 0.032 -->
@@ -53,6 +81,5 @@
                 <geometry name="ax12mesh">
                     <mesh
-                        filename="package://sf_dynamixel/defs/ax12_box_plain.stl"
-                        scale="0.001 0.001 0.001"/>
+                        filename="package://sf_dynamixel/meshes/ax12_box_plain.stl" scale="0.001 0.001 0.001"/>
                 </geometry>
                 <!-- xyz 0.050 0.038 0.032 -->

File: sf_dynamixel/defs/fp04_02.xacro (robot description, xacro)
@@ -14,5 +14,5 @@
                 <geometry name="fp04_02mesh">
                     <mesh
-                        filename="package://sf_dynamixel/defs/F2.stl"
+                        filename="package://sf_dynamixel/meshes/F2.stl"
                         scale="0.001 0.001 0.001"/>
                 </geometry>

Commit message: Fix sunflower next joints

File: sf_dynamixel/defs/dynamixel_ax12.xacro (robot description, xacro)
@@ -1,93 +1,88 @@
 <?xml version="1.0" encoding="UTF-8"?>
-<robot
-    xmlns:controller="http://playerstage.sourceforge.net/gazebo/xmlschema/#controller"
-    xmlns:interface="http://playerstage.sourceforge.net/gazebo/xmlschema/#interface"
-    xmlns:sensor="http://playerstage.sourceforge.net/gazebo/xmlschema/#sensor" xmlns:xacro="http://ros.org/wiki/xacro">
-    <xacro:macro name="ax12" params="name parent minPosition maxPosition maxVelocity">
-        <joint name="${name}_joint" type="revolute">
-            <parent link="${parent}_link"/>
-            <child link="${name}_link"/>
-            <origin xyz="0.0385 0 0" rpy="1.5707 0 0"/>
-            <axis xyz="0 0 1"/>
-            <limit effort="0" lower="${minPosition}"
-                upper="${maxPosition}" velocity="${maxVelocity}"/>
-        </joint>
-        <link name="${name}_link">
-            <collision>
-                <geometry>
-                    <box size="0.050 0.038 0.032"/>
-                </geometry>
-                <origin rpy="-1.5707 0 0" xyz="-0.0385 0 0"/>
-            </collision>
-            <visual>
-                <geometry name="ax12mesh">
-                    <mesh
-                        filename="package://sf_dynamixel/meshes/ax12_box_plain.stl" scale="0.001 0.001 0.001"/>
-                </geometry>
-                <!-- xyz 0.050 0.038 0.032 -->
-                <origin rpy="0 0 0" xyz="0.0135 0 0"/>
-                <material name="black_plastic">
-                    <color rgba="0.3 0.3 0.3 1"/>
-                </material>
-            </visual>
-        </link>
-    </xacro:macro>
-    <xacro:macro name="ax12old" params="name parent minPosition maxPosition maxVelocity *origin">
-        <joint name="${name}_joint" type="revolute">
-            <parent link="${parent}_link"/>
-            <child link="${name}_link"/>
-            <insert_block name="origin"/>
-            <axis xyz="0 -1 0"/>
-            <limit effort="0" lower="${minPosition}"
-                upper="${maxPosition}" velocity="${maxVelocity}"/>
-        </joint>
-        <link name="${name}_link">
-            <collision>
-                <geometry>
-                    <box size="0.050 0.038 0.032"/>
-                </geometry>
-                <origin rpy="0 0 0" xyz="0.0385 0 0"/>
-            </collision>
-            <visual>
-                <geometry name="ax12mesh">
-                    <mesh
-                        filename="package://sf_dynamixel/meshes/ax12_box_plain.stl" scale="0.001 0.001 0.001"/>
-                </geometry>
-                <!-- xyz 0.050 0.038 0.032 -->
-                <origin rpy="0 0 0" xyz="0.0135 0 0"/>
-                <material name="black_plastic">
-                    <color rgba="0.3 0.3 0.3 1"/>
-                </material>
-            </visual>
-        </link>
-    </xacro:macro>
-    <xacro:macro name="ax12inverted" params="name parent minPosition maxPosition maxVelocity *origin">
-        <joint name="${name}_joint" type="revolute">
-            <parent link="${parent}_link"/>
-            <child link="${name}_link"/>
-            <insert_block name="origin"/>
-            <axis xyz="-1 0 0"/>
-            <limit effort="0" lower="${minPosition}"
-                upper="${maxPosition}" velocity="${maxVelocity}"/>
-        </joint>
-        <link name="${name}_link">
-            <collision>
-                <geometry>
-                    <box size="0.050 0.038 0.032"/>
-                </geometry>
-                <origin rpy="0 0 1.5707" xyz="0.0385 0 0"/>
-            </collision>
-            <visual>
-                <geometry name="ax12mesh">
-                    <mesh
-                        filename="package://sf_dynamixel/meshes/ax12_box_plain.stl" scale="0.001 0.001 0.001"/>
-                </geometry>
-                <!-- xyz 0.050 0.038 0.032 -->
-                <origin rpy="0 0 0" xyz="0.0135 0 0"/>
-                <material name="black_plastic">
-                    <color rgba="0.3 0.3 0.3 1"/>
-                </material>
-            </visual>
-        </link>
-    </xacro:macro>
+<robot xmlns:controller="http://playerstage.sourceforge.net/gazebo/xmlschema/#controller"
+	xmlns:interface="http://playerstage.sourceforge.net/gazebo/xmlschema/#interface"
+	xmlns:sensor="http://playerstage.sourceforge.net/gazebo/xmlschema/#sensor"
+	xmlns:xacro="http://ros.org/wiki/xacro">
+	<xacro:macro name="ax12"
+		params="name parent minPosition maxPosition maxVelocity *origin">
+		<link name="${name}_box_link">
+			<visual>
+				<geometry name="ax12mesh">
+					<mesh filename="package://sf_dynamixel/meshes/ax12_box_plain.stl"
+						scale="0.001 0.001 0.001" />
+				</geometry>
+				<material name="plastic_black">
+					<color rgba="0.33 0.33 0.33 1" />
+				</material>
+				<origin rpy="-1.57075 1.57075 0" xyz="0 0 0.025" />
+			</visual>
+		</link>
+		<link name="${name}_link">
+			<visual>
+				<geometry>
+					<cylinder length="0.005" radius="0.011" />
+				</geometry>
+				<material name="plastic_white">
+					<color rgba="0.9 0.9 0.9 1" />
+				</material>
+				<origin rpy="0 1.57075 0" xyz="0.0025 0 0" />
+			</visual>
+		</link>
+		<joint name="${name}_joint" type="revolute">
+			<parent link="${name}_box_link" />
+			<child link="${name}_link" />
+			<origin xyz="0.0165 0 0.037" />
+			<axis xyz="1 0 0" />
+			<limit effort="0" lower="-1.5707" upper="1.5707" velocity="1" />
+		</joint>
+		<joint name="${name}_box_joint" type="fixed">
+			<parent link="${parent}_link" />
+			<child link="${name}_box_link" />
+			<insert_block name="origin" />
+		</joint>
+	</xacro:macro>
+	<xacro:macro name="ax12inverted"
+		params="name parent minPosition maxPosition maxVelocity *origin">
+		<link name="${name}_box_link">
+			<visual>
+				<geometry name="ax12mesh">
+					<mesh filename="package://sf_dynamixel/meshes/ax12_box_plain.stl"
+						scale="0.001 0.001 0.001" />
+				</geometry>
+				<material name="plastic_black">
+					<color rgba="0.33 0.33 0.33 1" />
+				</material>
+				<origin rpy="1.57075 0 3.14159" xyz="-0.012 0 0.019" />
+			</visual>
+		</link>
+		<link name="${name}_cyl_link">
+			<visual>
+				<geometry>
+					<cylinder length="0.005" radius="0.011" />
+				</geometry>
+				<material name="plastic_white">
+					<color rgba="0.9 0.9 0.9 1" />
+				</material>
+				<origin rpy="0 0 0" xyz="0 0 0.0025" />
+			</visual>
+		</link>
+		<link name="${name}_link"></link>
+		<joint name="${name}_box_joint" type="revolute">
+			<parent link="${name}_cyl_link" />
+			<child link="${name}_box_link" />
+			<origin xyz="0 0 0" />
+			<axis xyz="0 0 1" />
+			<limit effort="0" lower="-1.5707" upper="1.5707" velocity="1" />
+		</joint>
+		<joint name="${name}_cyl_joint" type="fixed">
+			<parent link="${parent}_link" />
+			<child link="${name}_cyl_link" />
+			<insert_block name="origin" />
+		</joint>
+		<joint name="{name}_joint" type="fixed">
+			<parent link="${name}_box_link" />
+			<child link="${name}_link" />
+			<origin xyz="0 0 0.038" />
+		</joint>
+	</xacro:macro>
 </robot>

File: sf_dynamixel/defs/fp04_02.xacro (robot description, xacro)
@@ -1,27 +1,30 @@
 <?xml version="1.0" encoding="UTF-8"?>
-<robot
-    xmlns:controller="http://playerstage.sourceforge.net/gazebo/xmlschema/#controller"
-    xmlns:interface="http://playerstage.sourceforge.net/gazebo/xmlschema/#interface"
-    xmlns:sensor="http://playerstage.sourceforge.net/gazebo/xmlschema/#sensor" xmlns:xacro="http://ros.org/wiki/xacro">
-    <xacro:macro name="fp04_02" params="name parent">
-        <joint name="${name}_joint" type="fixed">
-            <parent link="${parent}_link"/>
-            <child link="${name}_link"/>
-            <origin rpy="-1.5707 -1.5707 0" xyz="0.0014 0 0"/>
-        </joint>
-        <link name="${name}_link">
-            <visual>
-                <geometry name="fp04_02mesh">
-                    <mesh
-                        filename="package://sf_dynamixel/meshes/F2.stl"
-                        scale="0.001 0.001 0.001"/>
-                </geometry>
-                <!-- xyz 0.025 0.0485 0.0375 -->
-                <origin rpy="0 0 0" xyz="0 0 0"/>
-                <material name="green_plastic">
-                    <color rgba="0.1 0.8 0.3 1"/>
-                </material>
-            </visual>
-        </link>
-    </xacro:macro>
+<robot xmlns:controller="http://playerstage.sourceforge.net/gazebo/xmlschema/#controller"
+	xmlns:interface="http://playerstage.sourceforge.net/gazebo/xmlschema/#interface"
+	xmlns:sensor="http://playerstage.sourceforge.net/gazebo/xmlschema/#sensor"
+	xmlns:xacro="http://ros.org/wiki/xacro">
+	<xacro:macro name="fp04_02" params="name parent">
+		<link name="${name}_mesh_link">
+			<visual>
+				<geometry name="fp04_02mesh">
+					<mesh filename="package://sf_dynamixel/meshes/F2.stl" scale="0.001 0.001 0.001" />
+				</geometry>
+				<material name="plastic_green">
+					<color rgba="0.1 0.8 0.3 1" />
+				</material>
+				<origin rpy="-1.57075 0 1.57075" xyz="0 0 0.0" />
+			</visual>
+		</link>
+		<link name="${name}_link"></link>
+		<joint name="${name}_joint" type="fixed">
+			<parent link="${name}_mesh_link" />
+			<child link="${name}_link" />
+			<origin xyz="0 0 0.027" />
+		</joint>
+		<joint name="${name}_mesh_joint" type="fixed">
+			<parent link="${parent}_link" />
+			<child link="${name}_mesh_link" />
+			<origin xyz="-0.015 0 0" />
+		</joint>
+	</xacro:macro>
 </robot>

File: sf_robot/config/sf1-1.xacro (robot description, xacro)
@@ -34,5 +34,5 @@
 		</visual>
 	</link>
-    <!-- Override the 'continuous' joint from p3dx.xacro -->
+    <!-- Override the 'continuous' joint from p3dx.xacro which rviz doesn't support -->
     <joint name="base_swivel_joint_fixed" type="fixed">
         <origin xyz="-0.185 0 0.055" rpy="0 0 0"/>
@@ -88,5 +88,5 @@
                 name="neck_lower"
                 parent="${parent}"
-                minPosition="-1.5705"
+                minPosition="-1.5707"
                 maxPosition="1.5707"
                 maxVelocity="1">
@@ -100,8 +100,8 @@
                 name="neck_upper"
                 parent="neck_lower_hinge"
-                minPosition="-1.5705"
-                maxPosition="1.5707"
-                maxVelocity="1">
-            <origin rpy="1.5707 0 1.5707" xyz="0 -0.0635 0"/>
+                minPosition="-1.5707"
+                maxPosition="1.5707"
+                maxVelocity="1">
+            <origin rpy="0 0 0" xyz="0 0 0"/>
         </xacro:ax12>
         <xacro:fp04_02
@@ -109,11 +109,19 @@
                 parent="neck_upper">
         </xacro:fp04_02>
+        <xacro:ax12inverted
+                name="head_pan"
+                parent="neck_upper_hinge"
+                minPosition="-1.5705"
+                maxPosition="1.5707"
+                maxVelocity="1">
+            <origin rpy="0 0 0" xyz="0 0 0"/>
+        </xacro:ax12inverted>
         <xacro:ax12
                 name="head_tilt"
-                parent="neck_upper_hinge"
+                parent="head_pan"
                 minPosition="-1.5705"
                 maxPosition="1.5707"
                 maxVelocity="1">
-            <origin rpy="0 0 1.5707" xyz="0 -0.0635 0"/>
+            <origin rpy="0 0 0" xyz="0 0 0"/>
         </xacro:ax12>
         <xacro:fp04_02
@@ -121,15 +129,7 @@
                 parent="head_tilt">
         </xacro:fp04_02>
-        <xacro:ax12inverted
-                name="head_pan"
-                parent="head_tilt_hinge"
-                minPosition="-1.5705"
-                maxPosition="1.5707"
-                maxVelocity="1">
-            <origin rpy="0 0 1.5707" xyz="0 -0.0635 0"/>
-        </xacro:ax12inverted>
     </xacro:macro>
     <xacro:neck name="neck" parent="base">
-        <origin rpy="0 1.5707 0" xyz="0 0 0.79" />
+        <origin rpy="0 0 1.5707" xyz="0 0 0.75" />
     </xacro:neck>
 	<!-- Head -->
@@ -195,18 +195,22 @@
 	</xacro:macro>
 	<xacro:macro name="head" params="name parent *origin">
-		<joint name="${name}_joint" type="fixed">
-			<insert_block name="origin" />
-			<parent link="${parent}_link" />
-			<child link="${name}_link" />
+		<joint name="${name}_mount_joint" type="fixed">
+			<insert_block name="origin" />
+			<parent link="${parent}_link" />
+			<child link="${name}_mount_link" />
+		</joint>
+		<link name="${name}_mount_link"></link>
+		<joint name="${name}_joint" type="fixed">
+			<parent link="${name}_mount_link" />
+			<child link="${name}_link" />
+			<origin rpy="0 0 0 " xyz="0 0 -0.0475" />
 		</joint>
 		<link name="${name}_link">
 			<inertial>
 				<mass value="0.1" />
-				<origin xyz="0 0 -0.05" rpy="0 0 0" />
-				<inertia ixx="0.001" ixy="0.0" ixz="0.0" iyy="0.001" iyz="0.0"
-					izz="0.001" />
-			</inertial>
-			<visual>
-				<origin xyz="0 0 -0.05" rpy="0 0 0" />
+				<inertia ixx="0.001" ixy="0.0" ixz="0.0" iyy="0.001" iyz="0.0"
+					izz="0.001" />
+			</inertial>
+			<visual>
 				<geometry>
 					<cylinder length="0.10" radius="0.11" />
@@ -217,5 +221,4 @@
 			</visual>
 			<collision>
-				<origin xyz="0 0 -0.05" rpy="0 0 0" />
 				<geometry>
 					<cylinder length="0.10" radius="0.11" />
@@ -224,15 +227,15 @@
 		</link>
 		<xacro:eye name="eye_r" parent="${name}">
-			<origin rpy="0.23 1.57 0" xyz="0.12 -0.06 -0.05" />
+			<origin rpy="0.23 1.57 0" xyz="0.12 -0.06 0" />
 		</xacro:eye>
 		<xacro:eye name="eye_l" parent="${name}">
-			<origin rpy="-0.23 1.57 0" xyz="0.12 0.06 -0.05" />
+			<origin rpy="-0.23 1.57 0" xyz="0.12 0.06 0" />
 		</xacro:eye>
 		<xacro:camera name="camera" parent="${name}">
-			<origin rpy="0 1.57 0" xyz="0.11 0.00 -0.07" />
+			<origin rpy="0 1.57 0" xyz="0.11 0.00 -0.02" />
 		</xacro:camera>
 	</xacro:macro>
-	<xacro:head name="head" parent="head_pan">
-		<origin rpy="0 1.5707 3.14159" xyz="-0.05 0 0" />
+	<xacro:head name="head" parent="head_tilt_hinge">
+		<origin rpy="0 0 -1.5707" xyz="0 0 0" />
 	</xacro:head>
 	<!--Body -->

Commit message: fix joint name

File: sf_dynamixel/defs/dynamixel_ax12.xacro (robot description, xacro)
@@ -68,5 +68,5 @@
 		</link>
 		<link name="${name}_link"></link>
-		<joint name="${name}_box_joint" type="revolute">
+		<joint name="${name}_joint" type="revolute">
 			<parent link="${name}_cyl_link" />
 			<child link="${name}_box_link" />
@@ -80,5 +80,5 @@
 			<insert_block name="origin" />
 		</joint>
-		<joint name="{name}_joint" type="fixed">
+		<joint name="{name}_box_joint" type="fixed">
 			<parent link="${name}_box_link" />
 			<child link="${name}_link" />
