Commit message: Gazebo compatability changes

File: sf_dynamixel/defs/dynamixel_ax12.xacro (robot description, xacro)
@@ -17,4 +17,15 @@
 				<origin rpy="-1.57075 1.57075 0" xyz="0 0 0.025" />
 			</visual>
+			<inertial>
+				<mass value="0.01" />
+				<inertia ixx="0.001" ixy="0.0" ixz="0.0" iyy="0.001" iyz="0.0"
+					izz="0.001" />
+			</inertial>
+			<collision>
+				<geometry name="ax12mesh">
+					<mesh filename="package://sf_dynamixel/meshes/ax12_box_plain.stl"
+						scale="0.001 0.001 0.001" />
+				</geometry>
+			</collision>
 		</link>
 		<link name="${name}_link">
@@ -28,4 +39,14 @@
 				<origin rpy="0 1.57075 0" xyz="0.0025 0 0" />
 			</visual>
+			<inertial>
+				<mass value="0.001" />
+				<inertia ixx="0.001" ixy="0.0" ixz="0.0" iyy="0.001" iyz="0.0"
+					izz="0.001" />
+			</inertial>
+			<collision>
+				<geometry>
+					<cylinder length="0.005" radius="0.011" />
+				</geometry>
+			</collision>
 		</link>
 		<joint name="${name}_joint" type="revolute">
@@ -41,4 +62,10 @@
 			<insert_block name="origin" />
 		</joint>
+		<gazebo reference="${name}_box_link">
+			<material>Gazebo/FlatBlack</material>
+		</gazebo>
+		<gazebo reference="${name}_link">
+			<material>Gazebo/White</material>
+		</gazebo>
 	</xacro:macro>
 	<xacro:macro name="ax12inverted"
@@ -50,9 +77,20 @@
 						scale="0.001 0.001 0.001" />
 				</geometry>
-				<material name="plastic_black">
-					<color rgba="0.33 0.33 0.33 1" />
-				</material>
+				<material name="plastic_black" />
 				<origin rpy="1.57075 0 3.14159" xyz="-0.012 0 0.019" />
 			</visual>
+			<inertial>
+				<mass value="0.01" />
+				<origin rpy="0 0 0" xyz="-0.012 0 0.019" />
+				<inertia ixx="0.001" ixy="0.0" ixz="0.0" iyy="0.001" iyz="0.0"
+					izz="0.001" />
+			</inertial>
+			<collision>
+				<origin rpy="1.57075 0 3.14159" xyz="-0.012 0 0.019" />
+				<geometry name="ax12mesh">
+					<mesh filename="package://sf_dynamixel/meshes/ax12_box_plain.stl"
+						scale="0.001 0.001 0.001" />
+				</geometry>
+			</collision>
 		</link>
 		<link name="${name}_cyl_link">
@@ -61,9 +99,19 @@
 					<cylinder length="0.005" radius="0.011" />
 				</geometry>
-				<material name="plastic_white">
-					<color rgba="0.9 0.9 0.9 1" />
-				</material>
+				<material name="plastic_white" />
 				<origin rpy="0 0 0" xyz="0 0 0.0025" />
 			</visual>
+			<inertial>
+				<mass value="0.001" />
+				<inertia ixx="0.001" ixy="0.0" ixz="0.0" iyy="0.001" iyz="0.0"
+					izz="0.001" />
+				<origin rpy="0 0 0" xyz="0 0 0.0025" />
+			</inertial>
+			<collision>
+				<geometry>
+					<cylinder length="0.005" radius="0.011" />
+					<origin rpy="0 0 0" xyz="0 0 0.0025" />
+				</geometry>
+			</collision>
 		</link>
 		<link name="${name}_link"></link>
@@ -80,9 +128,15 @@
 			<insert_block name="origin" />
 		</joint>
-		<joint name="{name}_box_joint" type="fixed">
+		<joint name="${name}_box_joint" type="fixed">
 			<parent link="${name}_box_link" />
 			<child link="${name}_link" />
 			<origin xyz="0 0 0.038" />
 		</joint>
+		<gazebo reference="${name}_box_link">
+			<material>Gazebo/FlatBlack</material>
+		</gazebo>
+		<gazebo reference="${name}_cyl_link">
+			<material>Gazebo/White</material>
+		</gazebo>
 	</xacro:macro>
 </robot>

File: sf_dynamixel/defs/fp04_02.xacro (robot description, xacro)
@@ -15,4 +15,15 @@
 				<origin rpy="-1.57075 0 1.57075" xyz="0 0 0.0" />
 			</visual>
+			<collision>
+				<geometry name="fp04_02mesh">
+					<mesh filename="package://sf_dynamixel/meshes/F2.stl" scale="0.001 0.001 0.001" />
+				</geometry>
+			</collision>
+			<inertial>
+				<mass value="0.005" />
+				<inertia ixx="0.001" ixy="0.0" ixz="0.0" iyy="0.001" iyz="0.0"
+					izz="0.001" />
+				<origin rpy="0 0 0" xyz="0 0 0.0025" />
+			</inertial>
 		</link>
 		<link name="${name}_link"></link>
@@ -27,4 +38,7 @@
 			<origin xyz="-0.015 0 0" />
 		</joint>
+		<gazebo reference="${name}_mesh_link">
+			<material>Gazebo/Green</material>
+		</gazebo>
 	</xacro:macro>
 </robot>

File: sf_robot/config/hokuyo_laser.xacro (robot description, xacro)
@@ -1,7 +1,4 @@
 <?xml version="1.0"?>
-<robot xmlns:sensor="http://playerstage.sourceforge.net/gazebo/xmlschema/#sensor"
-	xmlns:controller="http://playerstage.sourceforge.net/gazebo/xmlschema/#controller"
-	xmlns:interface="http://playerstage.sourceforge.net/gazebo/xmlschema/#interface"
-	xmlns:xacro="http://ros.org/wiki/xacro">
+<robot xmlns:xacro="http://ros.org/wiki/xacro">
 	<xacro:macro name="hokuyo_04lx_laser_ug01"
 		params="name parent *origin ros_topic update_rate min_angle max_angle">
@@ -62,5 +59,5 @@
 			</collision>
 		</link>
-		<!--  Gazebo Config -->
+		<!-- Gazebo Config -->
 		<gazebo reference="${name}_link">
 			<sensor type="ray" name="${name}">
@@ -86,4 +83,5 @@
 				<plugin name="gazebo_ros_${name}_controller" filename="libgazebo_ros_laser.so">
 					<gaussianNoise>0.005</gaussianNoise>
+					<hokuyoMinIntensity>101</hokuyoMinIntensity>
 					<alwaysOn>true</alwaysOn>
 					<updateRate>${update_rate}</updateRate>
@@ -94,12 +92,8 @@
 		</gazebo>
 		<gazebo reference="${name}_link">
-			<material name="LaserBlack">
-				<color rgba="0.1 0.02 0.02 1.0" />
-			</material>
+			<material>Gazebo/FlatBlack</material>
 		</gazebo>
 		<gazebo reference="${name}_scan_link">
-			<material name="LaserBlack">
-				<color rgba="0.1 0.02 0.02 1.0" />
-			</material>
+			<material>Gazebo/FlatBlack</material>
 		</gazebo>
 	</xacro:macro>

File: sf_robot/config/sf1-1.xacro (robot description, xacro)
@@ -1,8 +1,4 @@
 <?xml version="1.0"?>
-<robot name="sf11"
-	xmlns:sensor="http://playerstage.sourceforge.net/gazebo/xmlschema/#sensor"
-	xmlns:controller="http://playerstage.sourceforge.net/gazebo/xmlschema/#controller"
-	xmlns:interface="http://playerstage.sourceforge.net/gazebo/xmlschema/#interface"
-	xmlns:xacro="http://ros.org/wiki/xacro">
+<robot name="sf11" xmlns:xacro="http://ros.org/wiki/xacro">
 	<!-- Base -->
 	<include filename="$(find p2os_urdf)/defs/pioneer3dx.xacro" />
@@ -22,8 +18,6 @@
 			<inertial>
 				<mass value="0.1" />
-				<origin xyz="0 0 0" />
 				<inertia ixx="1" ixy="0" ixz="0" iyy="1" iyz="0" izz="1" />
 			</inertial>
-			<origin rpy="0 0 0" xyz="0 0 0" />
 			<geometry name="top_geom">
 				<mesh filename="package://p2os_urdf/meshes/p3dx_meshes/top.stl" />
@@ -33,16 +27,25 @@
 			</material>
 		</visual>
+		<collision>
+			<geometry name="top_geom">
+				<mesh filename="package://p2os_urdf/meshes/p3dx_meshes/top.stl" />
+			</geometry>
+		</collision>
 	</link>
-    <!-- Override the 'continuous' joint from p3dx.xacro which rviz doesn't support -->
-    <joint name="base_swivel_joint_fixed" type="fixed">
-        <origin xyz="-0.185 0 0.055" rpy="0 0 0"/>
-        <parent link="base_link"/>
-        <child link="swivel"/>
-    </joint>
-    <joint name="swivel_hubcap_joint_fixed" type="fixed">
-        <origin xyz="-0.026 0 -0.016" rpy="0 0 0"/>
-        <parent link="swivel"/>
-        <child link="center_wheel"/>
-    </joint>
+	<gazebo reference="base_plate_joint">
+		<material>Gazebo/Wood</material>
+	</gazebo>
+	<!-- Override the 'continuous' joint from p3dx.xacro which rviz doesn't
+		support -->
+	<joint name="base_swivel_joint_fixed" type="fixed">
+		<origin xyz="-0.185 0 0.055" rpy="0 0 0" />
+		<parent link="base_link" />
+		<child link="swivel" />
+	</joint>
+	<joint name="swivel_hubcap_joint_fixed" type="fixed">
+		<origin xyz="-0.026 0 -0.016" rpy="0 0 0" />
+		<parent link="swivel" />
+		<child link="center_wheel" />
+	</joint>
 	<!-- Tray -->
 	<xacro:macro name="tray" params="name parent *origin">
@@ -51,16 +54,14 @@
 			<parent link="${parent}_link" />
 			<child link="${name}_link" />
-			<limit effort="0" lower="0.0" upper="0.15" velocity="0.5"/>
-			<axis xyz="1 0 0"/>
+			<limit effort="0" lower="0.0" upper="0.15" velocity="0.5" />
+			<axis xyz="1 0 0" />
 		</joint>
 		<link name="${name}_link">
 			<inertial>
 				<mass value="2" />
-				<origin xyz="0 0 0" rpy="0 0 0" />
-				<inertia ixx="0.001" ixy="0.0" ixz="0.0" iyy="0.001" iyz="0.0"
-					izz="0.001" />
-			</inertial>
-			<visual>
-				<origin xyz="0 0 0" rpy="0 0 0" />
+				<inertia ixx="0.001" ixy="0.0" ixz="0.0" iyy="0.001" iyz="0.0"
+					izz="0.001" />
+			</inertial>
+			<visual>
 				<geometry>
 					<box size="0.23 0.325 0.18" />
@@ -71,5 +72,4 @@
 			</visual>
 			<collision>
-				<origin xyz="0 0 0" rpy="0 0 0" />
 				<geometry>
 					<box size="0.23 0.325 0.18" />
@@ -77,60 +77,41 @@
 			</collision>
 		</link>
+		<gazebo reference="${name}_link">
+			<material>Gazebo/Wood</material>
+		</gazebo>
 	</xacro:macro>
 	<xacro:tray name="tray" parent="base">
 		<origin rpy="0 0 0" xyz="0.01 0 0.645" />
 	</xacro:tray>
-    <!-- Neck -->
-    <include filename="$(find sf_dynamixel)/defs/dynamixel_ax12.xacro" />
-    <include filename="$(find sf_dynamixel)/defs/fp04_02.xacro" />
-    <xacro:macro name="neck" params="name parent *origin">
-        <xacro:ax12
-                name="neck_lower"
-                parent="${parent}"
-                minPosition="-1.5707"
-                maxPosition="1.5707"
-                maxVelocity="1">
-            <insert_block name="origin"/>
-        </xacro:ax12>
-        <xacro:fp04_02
-                name="neck_lower_hinge"
-                parent="neck_lower">
-        </xacro:fp04_02>
-        <xacro:ax12
-                name="neck_upper"
-                parent="neck_lower_hinge"
-                minPosition="-1.5707"
-                maxPosition="1.5707"
-                maxVelocity="1">
-            <origin rpy="0 0 0" xyz="0 0 0"/>
-        </xacro:ax12>
-        <xacro:fp04_02
-                name="neck_upper_hinge"
-                parent="neck_upper">
-        </xacro:fp04_02>
-        <xacro:ax12inverted
-                name="head_pan"
-                parent="neck_upper_hinge"
-                minPosition="-1.5705"
-                maxPosition="1.5707"
-                maxVelocity="1">
-            <origin rpy="0 0 0" xyz="0 0 0"/>
-        </xacro:ax12inverted>
-        <xacro:ax12
-                name="head_tilt"
-                parent="head_pan"
-                minPosition="-1.5705"
-                maxPosition="1.5707"
-                maxVelocity="1">
-            <origin rpy="0 0 0" xyz="0 0 0"/>
-        </xacro:ax12>
-        <xacro:fp04_02
-                name="head_tilt_hinge"
-                parent="head_tilt">
-        </xacro:fp04_02>
-    </xacro:macro>
-    <xacro:neck name="neck" parent="base">
-        <origin rpy="0 0 1.5707" xyz="0 0 0.75" />
-    </xacro:neck>
+	<!-- Neck -->
+	<include filename="$(find sf_dynamixel)/defs/dynamixel_ax12.xacro" />
+	<include filename="$(find sf_dynamixel)/defs/fp04_02.xacro" />
+	<xacro:macro name="neck" params="name parent *origin">
+		<xacro:ax12 name="neck_lower" parent="${parent}"
+			minPosition="-1.5707" maxPosition="1.5707" maxVelocity="1">
+			<insert_block name="origin" />
+		</xacro:ax12>
+		<xacro:fp04_02 name="neck_lower_hinge" parent="neck_lower">
+		</xacro:fp04_02>
+		<xacro:ax12 name="neck_upper" parent="neck_lower_hinge"
+			minPosition="-1.5707" maxPosition="1.5707" maxVelocity="1">
+			<origin rpy="0 0 0" xyz="0 0 0" />
+		</xacro:ax12>
+		<xacro:fp04_02 name="neck_upper_hinge" parent="neck_upper">
+		</xacro:fp04_02>
+		<xacro:ax12inverted name="head_pan" parent="neck_upper_hinge"
+			minPosition="-1.5705" maxPosition="1.5707" maxVelocity="1">
+			<origin rpy="0 0 0" xyz="0 0 0" />
+		</xacro:ax12inverted>
+		<xacro:ax12 name="head_tilt" parent="head_pan" minPosition="-1.5705"
+			maxPosition="1.5707" maxVelocity="1">
+			<origin rpy="0 0 0" xyz="0 0 0" />
+		</xacro:ax12>
+		<xacro:fp04_02 name="head_tilt_hinge" parent="head_tilt">
+		</xacro:fp04_02>
+	</xacro:macro>
+	<xacro:neck name="neck" parent="base">
+		<origin rpy="0 0 1.5707" xyz="0 0 0.75" />
+	</xacro:neck>
 	<!-- Head -->
 	<xacro:macro name="camera" params="name parent *origin">
@@ -143,10 +124,8 @@
 			<inertial>
 				<mass value="0.01" />
-				<origin xyz="0 0 0" rpy="0 0 0" />
-				<inertia ixx="0.001" ixy="0.0" ixz="0.0" iyy="0.001" iyz="0.0"
-					izz="0.001" />
-			</inertial>
-			<visual>
-				<origin xyz="0 0 0" rpy="0 0 0" />
+				<inertia ixx="0.001" ixy="0.0" ixz="0.0" iyy="0.001" iyz="0.0"
+					izz="0.001" />
+			</inertial>
+			<visual>
 				<geometry>
 					<cylinder length="0.002" radius="0.015" />
@@ -157,5 +136,4 @@
 			</visual>
 			<collision>
-				<origin xyz="0 0 0" rpy="0 0 0" />
 				<geometry>
 					<cylinder length="0.002" radius="0.015" />
@@ -163,4 +141,7 @@
 			</collision>
 		</link>
+		<gazebo reference="${name}_link">
+			<material>Gazebo/Black</material>
+		</gazebo>
 	</xacro:macro>
 	<xacro:macro name="eye" params="name parent *origin">
@@ -173,10 +154,8 @@
 			<inertial>
 				<mass value="0.01" />
-				<origin xyz="0 0 0" rpy="0 0 0" />
-				<inertia ixx="0.001" ixy="0.0" ixz="0.0" iyy="0.001" iyz="0.0"
-					izz="0.001" />
-			</inertial>
-			<visual>
-				<origin xyz="0 0 0" rpy="0 0 0" />
+				<inertia ixx="0.001" ixy="0.0" ixz="0.0" iyy="0.001" iyz="0.0"
+					izz="0.001" />
+			</inertial>
+			<visual>
 				<geometry>
 					<cylinder length="0.015" radius="0.03" />
@@ -187,5 +166,4 @@
 			</visual>
 			<collision>
-				<origin xyz="0 0 0" rpy="0 0 0" />
 				<geometry>
 					<cylinder length="0.015" radius="0.03" />
@@ -193,4 +171,7 @@
 			</collision>
 		</link>
+		<gazebo reference="${name}_link">
+			<material>Gazebo/White</material>
+		</gazebo>
 	</xacro:macro>
 	<xacro:macro name="head" params="name parent *origin">
@@ -226,4 +207,7 @@
 			</collision>
 		</link>
+		<gazebo reference="${name}_link">
+			<material>Gazebo/Grey</material>
+		</gazebo>
 		<xacro:eye name="eye_r" parent="${name}">
 			<origin rpy="0.23 1.57 0" xyz="0.12 -0.06 0" />
@@ -269,4 +253,7 @@
 			</collision>
 		</link>
+		<gazebo reference="${name}_link">
+			<material>Gazebo/White</material>
+		</gazebo>
 	</xacro:macro>
 	<xacro:body name="body" parent="base">

Commit message: More gazebo changes

File: sf_dynamixel/defs/dynamixel_ax12.xacro (robot description, xacro)
@@ -62,4 +62,15 @@
 			<insert_block name="origin" />
 		</joint>
+		<transmission name="${name}_trans">
+			<type>transmission_interface/SimpleTransmission</type>
+			<joint name="${name}_joint">
+				<hardwareInterface>EffortJointInterface</hardwareInterface>
+			</joint>
+			<actuator name="${name}_motor">
+				<hardwareInterface>EffortJointInterface</hardwareInterface>
+				<mechanicalReduction>1</mechanicalReduction>
+			</actuator>
+		</transmission>
+		<!--  Gazebo Config -->
 		<gazebo reference="${name}_box_link">
 			<material>Gazebo/FlatBlack</material>
@@ -133,4 +144,15 @@
 			<origin xyz="0 0 0.038" />
 		</joint>
+		<transmission name="${name}_trans">
+			<type>transmission_interface/SimpleTransmission</type>
+			<joint name="${name}_joint">
+				<hardwareInterface>EffortJointInterface</hardwareInterface>
+			</joint>
+			<actuator name="${name}_motor">
+				<hardwareInterface>EffortJointInterface</hardwareInterface>
+				<mechanicalReduction>1</mechanicalReduction>
+			</actuator>
+		</transmission>
+		<!--  Gazebo Config -->
 		<gazebo reference="${name}_box_link">
 			<material>Gazebo/FlatBlack</material>

File: sf_dynamixel/defs/fp04_02.xacro (robot description, xacro)
@@ -1,4 +1,5 @@
 <?xml version="1.0" encoding="UTF-8"?>
-<robot xmlns:controller="http://playerstage.sourceforge.net/gazebo/xmlschema/#controller"
+<robot
+	xmlns:controller="http://playerstage.sourceforge.net/gazebo/xmlschema/#controller"
 	xmlns:interface="http://playerstage.sourceforge.net/gazebo/xmlschema/#interface"
 	xmlns:sensor="http://playerstage.sourceforge.net/gazebo/xmlschema/#sensor"

File: sf_robot/config/sf1-1.xacro (robot description, xacro)
@@ -1,4 +1,8 @@
 <?xml version="1.0"?>
-<robot name="sf11" xmlns:xacro="http://ros.org/wiki/xacro">
+<robot name="sf11"
+	xmlns:controller="http://playerstage.sourceforge.net/gazebo/xmlschema/#controller"
+	xmlns:interface="http://playerstage.sourceforge.net/gazebo/xmlschema/#interface"
+	xmlns:sensor="http://playerstage.sourceforge.net/gazebo/xmlschema/#sensor"
+	xmlns:xacro="http://ros.org/wiki/xacro">
 	<!-- Base -->
 	<include filename="$(find p2os_urdf)/defs/pioneer3dx.xacro" />
@@ -77,4 +81,15 @@
 			</collision>
 		</link>
+		<transmission name="${name}_trans">
+			<type>transmission_interface/SimpleTransmission</type>
+			<joint name="${name}_joint">
+				<hardwareInterface>EffortJointInterface</hardwareInterface>
+			</joint>
+			<actuator name="${name}_motor">
+				<hardwareInterface>EffortJointInterface</hardwareInterface>
+				<mechanicalReduction>1</mechanicalReduction>
+			</actuator>
+		</transmission>
+		<!-- Gazebo Config -->
 		<gazebo reference="${name}_link">
 			<material>Gazebo/Wood</material>
@@ -101,8 +116,8 @@
 		</xacro:fp04_02>
 		<xacro:ax12inverted name="head_pan" parent="neck_upper_hinge"
-			minPosition="-1.5705" maxPosition="1.5707" maxVelocity="1">
+			minPosition="-1.5707" maxPosition="1.5707" maxVelocity="1">
 			<origin rpy="0 0 0" xyz="0 0 0" />
 		</xacro:ax12inverted>
-		<xacro:ax12 name="head_tilt" parent="head_pan" minPosition="-1.5705"
+		<xacro:ax12 name="head_tilt" parent="head_pan" minPosition="-1.5707"
 			maxPosition="1.5707" maxVelocity="1">
 			<origin rpy="0 0 0" xyz="0 0 0" />
@@ -115,5 +130,5 @@
 	</xacro:neck>
 	<!-- Head -->
-	<xacro:macro name="camera" params="name parent *origin">
+	<xacro:macro name="simple_camera" params="name parent *origin">
 		<joint name="${name}_joint" type="fixed">
 			<insert_block name="origin" />
@@ -141,6 +156,42 @@
 			</collision>
 		</link>
+		<!-- Gazebo Config -->
 		<gazebo reference="${name}_link">
 			<material>Gazebo/Black</material>
+			<sensor type="camera" name="${name}_sensor">
+				<always_on>true</always_on>
+				<update_rate>25.0</update_rate>
+				<camera name="${name}_camera">
+					<horizontal_fov>1.3962634</horizontal_fov>
+					<image>
+						<width>640</width>
+						<height>480</height>
+						<format>R8G8B8</format>
+					</image>
+					<clip>
+						<near>0.1</near>
+						<far>100</far>
+					</clip>
+				</camera>
+				<plugin name="${name}_controller" filename="libgazebo_ros_camera.so">
+					<alwaysOn>true</alwaysOn>
+					<updateRate>25.0</updateRate>
+					<cameraName>${name}_camera</cameraName>
+					<imageTopicName>image_raw</imageTopicName>
+					<cameraInfoTopicName>camera_info</cameraInfoTopicName>
+					<frameName>${name}_link</frameName>
+					<hackBaseline>0.07</hackBaseline>
+					<distortionK1>0.0</distortionK1>
+					<distortionK2>0.0</distortionK2>
+					<distortionK3>0.0</distortionK3>
+					<distortionT1>0.0</distortionT1>
+					<distortionT2>0.0</distortionT2>
+					<CxPrime>0</CxPrime>
+					<Cx>0</Cx>
+					<Cy>0</Cy>
+					<focalLength>0</focalLength>
+				</plugin>
+			</sensor>
+			<turnGravityOff>true</turnGravityOff>
 		</gazebo>
 	</xacro:macro>
@@ -216,7 +267,7 @@
 			<origin rpy="-0.23 1.57 0" xyz="0.12 0.06 0" />
 		</xacro:eye>
-		<xacro:camera name="camera" parent="${name}">
+		<xacro:simple_camera name="camera" parent="${name}">
 			<origin rpy="0 1.57 0" xyz="0.11 0.00 -0.02" />
-		</xacro:camera>
+		</xacro:simple_camera>
 	</xacro:macro>
 	<xacro:head name="head" parent="head_tilt_hinge">
@@ -260,3 +311,16 @@
 		<origin rpy="0 0 0" xyz="-0.04 0 0.245" />
 	</xacro:body>
+	<gazebo>
+		<plugin name="p3d_base_controller" filename="libgazebo_ros_p3d.so">
+			<alwaysOn>true</alwaysOn>
+			<updateRate>100.0</updateRate>
+			<bodyName>base_link</bodyName>
+			<topicName>base_pose_ground_truth</topicName>
+			<gaussianNoise>0.01</gaussianNoise>
+			<frameName>map</frameName>
+			<xyzOffset>0 0 0</xyzOffset>
+			<rpyOffset>0 0 0</rpyOffset>
+		</plugin>
+		<canonicalBody>base_footprint</canonicalBody>
+	</gazebo>
 </robot>
