Commit message: Add gazebo sim initial support

File: sf_dynamixel/defs/dynamixel_ax12.xacro (robot description, xacro)
@@ -62,15 +62,13 @@
 			<insert_block name="origin" />
 		</joint>
+		<!--  Gazebo Config -->
 		<transmission name="${name}_trans">
 			<type>transmission_interface/SimpleTransmission</type>
-			<joint name="${name}_joint">
-				<hardwareInterface>EffortJointInterface</hardwareInterface>
-			</joint>
+			<joint name="${name}_joint" />
 			<actuator name="${name}_motor">
-				<hardwareInterface>EffortJointInterface</hardwareInterface>
+				<hardwareInterface>PositionJointInterface</hardwareInterface>
 				<mechanicalReduction>1</mechanicalReduction>
 			</actuator>
 		</transmission>
-		<!--  Gazebo Config -->
 		<gazebo reference="${name}_box_link">
 			<material>Gazebo/FlatBlack</material>
@@ -144,15 +142,13 @@
 			<origin xyz="0 0 0.038" />
 		</joint>
+		<!--  Gazebo Config -->
 		<transmission name="${name}_trans">
 			<type>transmission_interface/SimpleTransmission</type>
-			<joint name="${name}_joint">
-				<hardwareInterface>EffortJointInterface</hardwareInterface>
-			</joint>
+			<joint name="${name}_joint" />
 			<actuator name="${name}_motor">
-				<hardwareInterface>EffortJointInterface</hardwareInterface>
+				<hardwareInterface>PositionJointInterface</hardwareInterface>
 				<mechanicalReduction>1</mechanicalReduction>
 			</actuator>
 		</transmission>
-		<!--  Gazebo Config -->
 		<gazebo reference="${name}_box_link">
 			<material>Gazebo/FlatBlack</material>

File: sf_robot/config/sf1-1.xacro (robot description, xacro)
@@ -1,14 +1,10 @@
 <?xml version="1.0"?>
-<robot name="sf11"
-	xmlns:controller="http://playerstage.sourceforge.net/gazebo/xmlschema/#controller"
-	xmlns:interface="http://playerstage.sourceforge.net/gazebo/xmlschema/#interface"
-	xmlns:sensor="http://playerstage.sourceforge.net/gazebo/xmlschema/#sensor"
-	xmlns:xacro="http://ros.org/wiki/xacro">
+<robot name="sf11" xmlns:controller="http://playerstage.sourceforge.net/gazebo/xmlschema/#controller" xmlns:interface="http://playerstage.sourceforge.net/gazebo/xmlschema/#interface"
+	xmlns:sensor="http://playerstage.sourceforge.net/gazebo/xmlschema/#sensor" xmlns:xacro="http://ros.org/wiki/xacro">
 	<!-- Base -->
 	<xacro:include filename="$(find p2os_urdf)/defs/pioneer3dx.xacro" />
 	<xacro:include filename="$(find sf_robot)/config/hokuyo_laser.xacro" />
-	<xacro:hokuyo_04lx_laser_ug01 name="base_laser_front"
-		parent="base" ros_topic="scan_front" update_rate="10" min_angle="-2.094"
-		max_angle="2.094">
+	<xacro:hokuyo_04lx_laser_ug01 name="base_laser_front" parent="base" ros_topic="scan_front" update_rate="10"
+		min_angle="-2.094" max_angle="2.094">
 		<origin rpy="0 0 0" xyz="0.15 0.0 0.245" />
 	</xacro:hokuyo_04lx_laser_ug01>
@@ -40,6 +36,5 @@
 		<material>Gazebo/Wood</material>
 	</gazebo>
-	<!-- Override the 'continuous' joint from p3dx.xacro which rviz doesn't
-		support -->
+	<!-- Override the 'continuous' joint from p3dx.xacro which rviz doesn't support -->
 	<joint name="base_swivel_joint_fixed" type="fixed">
 		<origin xyz="-0.185 0 0.055" rpy="0 0 0" />
@@ -64,6 +59,5 @@
 			<inertial>
 				<mass value="2" />
-				<inertia ixx="0.001" ixy="0.0" ixz="0.0" iyy="0.001" iyz="0.0"
-					izz="0.001" />
+				<inertia ixx="0.001" ixy="0.0" ixz="0.0" iyy="0.001" iyz="0.0" izz="0.001" />
 			</inertial>
 			<visual>
@@ -83,9 +77,7 @@
 		<transmission name="${name}_trans">
 			<type>transmission_interface/SimpleTransmission</type>
-			<joint name="${name}_joint">
-				<hardwareInterface>EffortJointInterface</hardwareInterface>
-			</joint>
+			<joint name="${name}_joint" />
 			<actuator name="${name}_motor">
-				<hardwareInterface>EffortJointInterface</hardwareInterface>
+				<hardwareInterface>PositionJointInterface</hardwareInterface>
 				<mechanicalReduction>1</mechanicalReduction>
 			</actuator>
@@ -103,22 +95,18 @@
 	<xacro:include filename="$(find sf_dynamixel)/defs/fp04_02.xacro" />
 	<xacro:macro name="neck" params="name parent *origin">
-		<xacro:ax12 name="neck_lower" parent="${parent}"
-			minPosition="-1.5707" maxPosition="1.5707" maxVelocity="1">
+		<xacro:ax12 name="neck_lower" parent="${parent}" minPosition="-1.5707" maxPosition="1.5707" maxVelocity="1">
 			<insert_block name="origin" />
 		</xacro:ax12>
 		<xacro:fp04_02 name="neck_lower_hinge" parent="neck_lower">
 		</xacro:fp04_02>
-		<xacro:ax12 name="neck_upper" parent="neck_lower_hinge"
-			minPosition="-1.5707" maxPosition="1.5707" maxVelocity="1">
+		<xacro:ax12 name="neck_upper" parent="neck_lower_hinge" minPosition="-1.5707" maxPosition="1.5707" maxVelocity="1">
 			<origin rpy="0 0 0" xyz="0 0 0" />
 		</xacro:ax12>
 		<xacro:fp04_02 name="neck_upper_hinge" parent="neck_upper">
 		</xacro:fp04_02>
-		<xacro:ax12inverted name="head_pan" parent="neck_upper_hinge"
-			minPosition="-1.5707" maxPosition="1.5707" maxVelocity="1">
+		<xacro:ax12inverted name="head_pan" parent="neck_upper_hinge" minPosition="-1.5707" maxPosition="1.5707" maxVelocity="1">
 			<origin rpy="0 0 -1.57079" xyz="0 0 0" />
 		</xacro:ax12inverted>
-		<xacro:ax12 name="head_tilt" parent="head_pan" minPosition="-1.5707"
-			maxPosition="1.5707" maxVelocity="1">
+		<xacro:ax12 name="head_tilt" parent="head_pan" minPosition="-1.5707" maxPosition="1.5707" maxVelocity="1">
 			<origin rpy="0 0 0" xyz="0 0 0" />
 		</xacro:ax12>
@@ -139,6 +127,5 @@
 			<inertial>
 				<mass value="0.01" />
-				<inertia ixx="0.001" ixy="0.0" ixz="0.0" iyy="0.001" iyz="0.0"
-					izz="0.001" />
+				<inertia ixx="0.001" ixy="0.0" ixz="0.0" iyy="0.001" iyz="0.0" izz="0.001" />
 			</inertial>
 			<visual>
@@ -205,6 +192,5 @@
 			<inertial>
 				<mass value="0.01" />
-				<inertia ixx="0.001" ixy="0.0" ixz="0.0" iyy="0.001" iyz="0.0"
-					izz="0.001" />
+				<inertia ixx="0.001" ixy="0.0" ixz="0.0" iyy="0.001" iyz="0.0" izz="0.001" />
 			</inertial>
 			<visual>
@@ -241,6 +227,5 @@
 			<inertial>
 				<mass value="0.1" />
-				<inertia ixx="0.001" ixy="0.0" ixz="0.0" iyy="0.001" iyz="0.0"
-					izz="0.001" />
+				<inertia ixx="0.001" ixy="0.0" ixz="0.0" iyy="0.001" iyz="0.0" izz="0.001" />
 			</inertial>
 			<visual>
@@ -285,6 +270,5 @@
 				<mass value="10" />
 				<origin xyz="0 0 0.2525" rpy="0 0 0" />
-				<inertia ixx="0.001" ixy="0.0" ixz="0.0" iyy="0.001" iyz="0.0"
-					izz="0.001" />
+				<inertia ixx="0.001" ixy="0.0" ixz="0.0" iyy="0.001" iyz="0.0" izz="0.001" />
 			</inertial>
 			<visual>
@@ -312,4 +296,7 @@
 	</xacro:body>
 	<gazebo>
+		<plugin name="gazebo_ros_control" filename="libgazebo_ros_control.so">
+			<robotNamespace>/sunflower1_1</robotNamespace>
+		</plugin>
 		<plugin name="p3d_base_controller" filename="libgazebo_ros_p3d.so">
 			<alwaysOn>true</alwaysOn>

Commit message: further work on a functional gazebo sim

File: sf_dynamixel/defs/dynamixel_ax12.xacro (robot description, xacro)
@@ -62,8 +62,10 @@
 			<insert_block name="origin" />
 		</joint>
-		<!--  Gazebo Config -->
+		<!-- Gazebo Config -->
 		<transmission name="${name}_trans">
 			<type>transmission_interface/SimpleTransmission</type>
-			<joint name="${name}_joint" />
+			<joint name="${name}_joint">
+				<hardwareInterface>PositionJointInterface</hardwareInterface>
+			</joint>
 			<actuator name="${name}_motor">
 				<hardwareInterface>PositionJointInterface</hardwareInterface>
@@ -142,8 +144,10 @@
 			<origin xyz="0 0 0.038" />
 		</joint>
-		<!--  Gazebo Config -->
+		<!-- Gazebo Config -->
 		<transmission name="${name}_trans">
 			<type>transmission_interface/SimpleTransmission</type>
-			<joint name="${name}_joint" />
+			<joint name="${name}_joint">
+				<hardwareInterface>PositionJointInterface</hardwareInterface>
+			</joint>
 			<actuator name="${name}_motor">
 				<hardwareInterface>PositionJointInterface</hardwareInterface>

File: sf_robot_description/config/hokuyo_laser.xacro (robot description, xacro)
@@ -31,4 +31,7 @@
 			</collision>
 		</link>
+		<gazebo reference="${name}_link">
+			<material>Gazebo/FlatBlack</material>
+		</gazebo>
 		<joint name="${name}_scan_joint" type="fixed">
 			<origin xyz="0 0 0.041" rpy="0 0 0" />
@@ -61,9 +64,8 @@
 		<!-- Gazebo Config -->
 		<gazebo reference="${name}_link">
-			<sensor type="ray" name="${name}">
-				<always_on>true</always_on>
-				<update_rate>${update_rate}</update_rate>
+			<sensor type="gpu_ray" name="${name}">
 				<pose>0 0 0 0 0 0</pose>
 				<visualize>false</visualize>
+				<update_rate>${update_rate}</update_rate>
 				<ray>
 					<scan>
@@ -81,9 +83,8 @@
 					</range>
 				</ray>
-				<plugin name="gazebo_ros_${name}_controller" filename="libgazebo_ros_laser.so">
+				<plugin name="gazebo_ros_${name}_controller" filename="libgazebo_ros_gpu_laser.so">
 					<gaussianNoise>0.005</gaussianNoise>
 					<hokuyoMinIntensity>101</hokuyoMinIntensity>
 					<alwaysOn>true</alwaysOn>
-					<updateRate>${update_rate}</updateRate>
 					<topicName>${ros_topic}</topicName>
 					<frameName>${name}_link</frameName>
@@ -91,10 +92,4 @@
 			</sensor>
 		</gazebo>
-		<gazebo reference="${name}_link">
-			<material>Gazebo/FlatBlack</material>
-		</gazebo>
-		<gazebo reference="${name}_scan_link">
-			<material>Gazebo/FlatBlack</material>
-		</gazebo>
 	</xacro:macro>
 </robot>

File: sf_robot_description/config/sf1-1.xacro (robot description, xacro)
@@ -1,12 +1,13 @@
 <?xml version="1.0"?>
-<robot name="sf11" xmlns:controller="http://playerstage.sourceforge.net/gazebo/xmlschema/#controller" xmlns:interface="http://playerstage.sourceforge.net/gazebo/xmlschema/#interface"
-	xmlns:sensor="http://playerstage.sourceforge.net/gazebo/xmlschema/#sensor" xmlns:xacro="http://ros.org/wiki/xacro">
+<robot name="sf11"
+	xmlns:controller="http://playerstage.sourceforge.net/gazebo/xmlschema/#controller"
+	xmlns:interface="http://playerstage.sourceforge.net/gazebo/xmlschema/#interface"
+	xmlns:sensor="http://playerstage.sourceforge.net/gazebo/xmlschema/#sensor"
+	xmlns:xacro="http://ros.org/wiki/xacro">
+	<xacro:include filename="$(find sf_robot_description)/config/hokuyo_laser.xacro" />
+	<xacro:include filename="$(find sf_dynamixel)/defs/dynamixel_ax12.xacro" />
+	<xacro:include filename="$(find sf_dynamixel)/defs/fp04_02.xacro" />
 	<!-- Base -->
-	<xacro:include filename="$(find p2os_urdf)/defs/pioneer3dx.xacro" />
-	<xacro:include filename="$(find sf_robot_desc)/config/hokuyo_laser.xacro" />
-	<xacro:hokuyo_04lx_laser_ug01 name="base_laser_front" parent="base" ros_topic="scan_front" update_rate="10"
-		min_angle="-2.094" max_angle="2.094">
-		<origin rpy="0 0 0" xyz="0.15 0.0 0.245" />
-	</xacro:hokuyo_04lx_laser_ug01>
+	<xacro:include filename="$(find sf_robot_description)/config/pioneer3dx.xacro" />
 	<joint name="base_plate_joint" type="fixed">
 		<origin rpy="0 0 0" xyz="0 0 0.0085" />
@@ -33,18 +34,7 @@
 		</collision>
 	</link>
-	<gazebo reference="base_plate_joint">
+	<gazebo reference="base_plate_link">
 		<material>Gazebo/Wood</material>
 	</gazebo>
-	<!-- Override the 'continuous' joint from p3dx.xacro which rviz doesn't support -->
-	<joint name="base_swivel_joint_fixed" type="fixed">
-		<origin xyz="-0.185 0 0.055" rpy="0 0 0" />
-		<parent link="base_link" />
-		<child link="swivel" />
-	</joint>
-	<joint name="swivel_hubcap_joint_fixed" type="fixed">
-		<origin xyz="-0.026 0 -0.016" rpy="0 0 0" />
-		<parent link="swivel" />
-		<child link="center_wheel" />
-	</joint>
 	<!-- Tray -->
 	<xacro:macro name="tray" params="name parent *origin">
@@ -59,5 +49,6 @@
 			<inertial>
 				<mass value="2" />
-				<inertia ixx="0.001" ixy="0.0" ixz="0.0" iyy="0.001" iyz="0.0" izz="0.001" />
+				<inertia ixx="0.001" ixy="0.0" ixz="0.0" iyy="0.001" iyz="0.0"
+					izz="0.001" />
 			</inertial>
 			<visual>
@@ -77,5 +68,7 @@
 		<transmission name="${name}_trans">
 			<type>transmission_interface/SimpleTransmission</type>
-			<joint name="${name}_joint" />
+			<joint name="${name}_joint">
+				<hardwareInterface>PositionJointInterface</hardwareInterface>
+			</joint>
 			<actuator name="${name}_motor">
 				<hardwareInterface>PositionJointInterface</hardwareInterface>
@@ -88,25 +81,24 @@
 		</gazebo>
 	</xacro:macro>
-	<xacro:tray name="tray" parent="base">
-		<origin rpy="0 0 0" xyz="0.01 0 0.645" />
-	</xacro:tray>
 	<!-- Neck -->
-	<xacro:include filename="$(find sf_dynamixel)/defs/dynamixel_ax12.xacro" />
-	<xacro:include filename="$(find sf_dynamixel)/defs/fp04_02.xacro" />
 	<xacro:macro name="neck" params="name parent *origin">
-		<xacro:ax12 name="neck_lower" parent="${parent}" minPosition="-1.5707" maxPosition="1.5707" maxVelocity="1">
+		<xacro:ax12 name="neck_lower" parent="${parent}"
+			minPosition="-1.5707" maxPosition="1.5707" maxVelocity="1">
 			<insert_block name="origin" />
 		</xacro:ax12>
 		<xacro:fp04_02 name="neck_lower_hinge" parent="neck_lower">
 		</xacro:fp04_02>
-		<xacro:ax12 name="neck_upper" parent="neck_lower_hinge" minPosition="-1.5707" maxPosition="1.5707" maxVelocity="1">
+		<xacro:ax12 name="neck_upper" parent="neck_lower_hinge"
+			minPosition="-1.5707" maxPosition="1.5707" maxVelocity="1">
 			<origin rpy="0 0 0" xyz="0 0 0" />
 		</xacro:ax12>
 		<xacro:fp04_02 name="neck_upper_hinge" parent="neck_upper">
 		</xacro:fp04_02>
-		<xacro:ax12inverted name="head_pan" parent="neck_upper_hinge" minPosition="-1.5707" maxPosition="1.5707" maxVelocity="1">
+		<xacro:ax12inverted name="head_pan" parent="neck_upper_hinge"
+			minPosition="-1.5707" maxPosition="1.5707" maxVelocity="1">
 			<origin rpy="0 0 -1.57079" xyz="0 0 0" />
 		</xacro:ax12inverted>
-		<xacro:ax12 name="head_tilt" parent="head_pan" minPosition="-1.5707" maxPosition="1.5707" maxVelocity="1">
+		<xacro:ax12 name="head_tilt" parent="head_pan" minPosition="-1.5707"
+			maxPosition="1.5707" maxVelocity="1">
 			<origin rpy="0 0 0" xyz="0 0 0" />
 		</xacro:ax12>
@@ -114,7 +106,4 @@
 		</xacro:fp04_02>
 	</xacro:macro>
-	<xacro:neck name="neck" parent="base">
-		<origin rpy="0 0 1.5707" xyz="0 0 0.75" />
-	</xacro:neck>
 	<!-- Head -->
 	<xacro:macro name="simple_camera" params="name parent *origin">
@@ -127,5 +116,6 @@
 			<inertial>
 				<mass value="0.01" />
-				<inertia ixx="0.001" ixy="0.0" ixz="0.0" iyy="0.001" iyz="0.0" izz="0.001" />
+				<inertia ixx="0.001" ixy="0.0" ixz="0.0" iyy="0.001" iyz="0.0"
+					izz="0.001" />
 			</inertial>
 			<visual>
@@ -192,5 +182,6 @@
 			<inertial>
 				<mass value="0.01" />
-				<inertia ixx="0.001" ixy="0.0" ixz="0.0" iyy="0.001" iyz="0.0" izz="0.001" />
+				<inertia ixx="0.001" ixy="0.0" ixz="0.0" iyy="0.001" iyz="0.0"
+					izz="0.001" />
 			</inertial>
 			<visual>
@@ -227,5 +218,6 @@
 			<inertial>
 				<mass value="0.1" />
-				<inertia ixx="0.001" ixy="0.0" ixz="0.0" iyy="0.001" iyz="0.0" izz="0.001" />
+				<inertia ixx="0.001" ixy="0.0" ixz="0.0" iyy="0.001" iyz="0.0"
+					izz="0.001" />
 			</inertial>
 			<visual>
@@ -256,58 +248,59 @@
 		</xacro:simple_camera>
 	</xacro:macro>
+	<!--Body -->
+	<xacro:macro name="body" params="name parent *origin">
+		<joint name="${name}_joint" type="fixed">
+			<insert_block name="origin" />
+			<parent link="${parent}_link" />
+			<child link="${name}_link" />
+		</joint>
+		<link name="${name}_link">
+			<inertial>
+				<mass value="10" />
+				<origin xyz="0 0 0.2525" rpy="0 0 0" />
+				<inertia ixx="0.001" ixy="0.0" ixz="0.0" iyy="0.001" iyz="0.0"
+					izz="0.001" />
+			</inertial>
+			<visual>
+				<origin xyz="0 0 0.2525" rpy="0 0 0" />
+				<geometry>
+					<box size="0.30 0.33 0.505" />
+				</geometry>
+				<material name="white">
+					<color rgba="0.98 0.98 0.90 1.0" />
+				</material>
+			</visual>
+			<collision>
+				<origin xyz="0 0 0.2525" rpy="0 0 0" />
+				<geometry>
+					<box size="0.30 0.33 0.505" />
+				</geometry>
+			</collision>
+		</link>
+		<gazebo reference="${name}_link">
+			<material>Gazebo/White</material>
+		</gazebo>
+	</xacro:macro>
 	<xacro:head name="head" parent="head_tilt_hinge">
 		<origin rpy="0 0 0" xyz="0 0 0" />
 	</xacro:head>
-	<!--Body -->
-	<xacro:macro name="body" params="name parent *origin">
-		<joint name="${name}_joint" type="fixed">
-			<insert_block name="origin" />
-			<parent link="${parent}_link" />
-			<child link="${name}_link" />
-		</joint>
-		<link name="${name}_link">
-			<inertial>
-				<mass value="10" />
-				<origin xyz="0 0 0.2525" rpy="0 0 0" />
-				<inertia ixx="0.001" ixy="0.0" ixz="0.0" iyy="0.001" iyz="0.0" izz="0.001" />
-			</inertial>
-			<visual>
-				<origin xyz="0 0 0.2525" rpy="0 0 0" />
-				<geometry>
-					<box size="0.30 0.33 0.505" />
-				</geometry>
-				<material name="white">
-					<color rgba="0.98 0.98 0.90 1.0" />
-				</material>
-			</visual>
-			<collision>
-				<origin xyz="0 0 0.2525" rpy="0 0 0" />
-				<geometry>
-					<box size="0.30 0.33 0.505" />
-				</geometry>
-			</collision>
-		</link>
-		<gazebo reference="${name}_link">
-			<material>Gazebo/White</material>
-		</gazebo>
-	</xacro:macro>
+	<xacro:tray name="tray" parent="base">
+		<origin rpy="0 0 0" xyz="0.01 0 0.645" />
+	</xacro:tray>
+	<xacro:neck name="neck" parent="base">
+		<origin rpy="0 0 1.5707" xyz="0 0 0.75" />
+	</xacro:neck>
 	<xacro:body name="body" parent="base">
 		<origin rpy="0 0 0" xyz="-0.04 0 0.245" />
 	</xacro:body>
+	<xacro:hokuyo_04lx_laser_ug01 name="base_laser_front"
+		parent="base" ros_topic="scan_front" update_rate="10" min_angle="-2.094"
+		max_angle="2.094">
+		<origin rpy="0 0 0" xyz="0.15 0.0 0.245" />
+	</xacro:hokuyo_04lx_laser_ug01>
 	<gazebo>
 		<plugin name="gazebo_ros_control" filename="libgazebo_ros_control.so">
 			<robotNamespace>/sunflower1_1</robotNamespace>
 		</plugin>
-		<plugin name="p3d_base_controller" filename="libgazebo_ros_p3d.so">
-			<alwaysOn>true</alwaysOn>
-			<updateRate>100.0</updateRate>
-			<bodyName>base_link</bodyName>
-			<topicName>base_pose_ground_truth</topicName>
-			<gaussianNoise>0.01</gaussianNoise>
-			<frameName>map</frameName>
-			<xyzOffset>0 0 0</xyzOffset>
-			<rpyOffset>0 0 0</rpyOffset>
-		</plugin>
-		<canonicalBody>base_footprint</canonicalBody>
 	</gazebo>
 </robot>
