Commit message: Reuse laser for person_sim, add gazebo plugins to person_sim

File: sf_robot_description/config/pioneer3dx.xacro (robot description, xacro)
@@ -5,6 +5,6 @@
 	xmlns:interface="http://playerstage.sourceforge.net/gazebo/xmlschema/#interface"
 	xmlns:xacro="http://ros.org/wiki/xacro">
-	<include filename="$(find sf_robot_description)/config/pioneer3dx_wheel.xacro" />
-	<include filename="$(find sf_robot_description)/config/pioneer3dx_sonar.xacro" />
+	<xacro:include filename="$(find sf_robot_description)/config/pioneer3dx_wheel.xacro" />
+	<xacro:include filename="$(find sf_robot_description)/config/pioneer3dx_sonar.xacro" />
 	<!-- Chassis -->
 	<link name="base_link">

File: simulation/person_sim/config/person.xacro (robot description, xacro)
@@ -5,6 +5,54 @@
 	xmlns:sensor="http://playerstage.sourceforge.net/gazebo/xmlschema/#sensor"
 	xmlns:xacro="http://ros.org/wiki/xacro">
+	<xacro:include filename="$(find sf_robot_description)/config/hokuyo_laser.xacro" />
 	<link name="base_link">
 	</link>
+	<xacro:macro name="wheel" params="name parent reflect *origin">
+		<link name="${parent}_${name}_wheel">
+			<inertial>
+				<mass value="0.5" />
+				<origin xyz="0 0 0" rpy="${-3.1415927/2} 0 0" />
+				<inertia ixx="0.012411765597" ixy="0" ixz="0" iyy="0.015218160428"
+					iyz="0" izz="0.011763977943" />
+			</inertial>
+			<visual name="${parent}_${name}_wheel_visual">
+				<origin xyz="0 0 0" rpy="${-3.1415927/2} 0 0" />
+				<geometry name="${parent}_${name}_wheel_geom">
+					<cylinder radius="0.1" length="0.02" />
+				</geometry>
+				<material name="WheelBlack">
+					<color rgba="0.117 0.117 0.117 1" />
+				</material>
+			</visual>
+			<collision>
+				<origin xyz="0 0 0" rpy="${-3.1415927/2} 0 0" />
+				<geometry name="${parent}_${name}_wheel_geom">
+					<cylinder radius="0.1" length="0.02" />
+				</geometry>
+			</collision>
+		</link>
+		<gazebo reference="${parent}_${name}_wheel">
+			<material value="Gazebo/Black" />
+		</gazebo>
+		<joint name="${parent}_${name}_wheel_joint" type="continuous">
+			<axis xyz="0 1 0" />
+			<anchor xyz="0 0 0" />
+			<limit effort="100" velocity="100" />
+			<dynamics damping="0.0" friction="0.0" />
+			<insert_block name="origin" />
+			<parent link="${parent}_link" />
+			<child link="${parent}_${name}_wheel" />
+		</joint>
+		<transmission name="${parent}_${name}_wheel_trans">
+			<type>transmission_interface/SimpleTransmission</type>
+			<joint name="${parent}_${name}_wheel_joint">
+				<hardwareInterface>EffortJointInterface</hardwareInterface>
+			</joint>
+			<actuator name="${parent}_${name}_wheel_motor">
+				<hardwareInterface>EffortJointInterface</hardwareInterface>
+				<mechanicalReduction>${reflect * (624/35) * (80/19)}</mechanicalReduction>
+			</actuator>
+		</transmission>
+	</xacro:macro>
 	<xacro:macro name="torso" params="name parent *origin">
 		<joint name="${name}_joint" type="fixed">
@@ -197,5 +245,4 @@
 		</gazebo>
 	</xacro:macro>
-	<xacro:include filename="$(find person_sim)/config/hokuyo_laser.xacro" />
 	<xacro:hokuyo_04lx_laser_ug01 name="base_laser_front"
 		parent="base" ros_topic="scan_front" update_rate="10" min_angle="-2.094"
@@ -217,3 +264,31 @@
 		<origin rpy="0 0 0" xyz="0 0.1 0" />
 	</xacro:leg>
+	<xacro:wheel name="front_right" parent="base" reflect="1">
+		<origin rpy="0 0 0" xyz=" -0.1 0.18 0" />
+	</xacro:wheel>
+	<xacro:wheel name="rear_right" parent="base" reflect="1">
+		<origin rpy="0 0 0" xyz="0.1 0.18 0" />
+	</xacro:wheel>
+	<xacro:wheel name="front_left" parent="base" reflect="-1">
+		<origin rpy="0 0 0" xyz="-0.1 -0.18 0" />
+	</xacro:wheel>
+	<xacro:wheel name="rear_left" parent="base" reflect="-1">
+		<origin rpy="0 0 0" xyz=" 0.1 -0.18 0" />
+	</xacro:wheel>
+	<gazebo>
+		<plugin name="skid_steer_drive_controller" filename="libgazebo_ros_skid_steer_drive.so">
+			<updateRate>100.0</updateRate>
+			<robotNamespace>/</robotNamespace>
+			<leftFrontJoint>base_front_left_wheel_joint</leftFrontJoint>
+			<rightFrontJoint>base_front_right_wheel_joint</rightFrontJoint>
+			<leftRearJoint>base_back_left_wheel_joint</leftRearJoint>
+			<rightRearJoint>base_back_right_wheel_joint</rightRearJoint>
+			<wheelSeparation>0.4</wheelSeparation>
+			<wheelDiameter>0.215</wheelDiameter>
+			<robotBaseFrame>base_link</robotBaseFrame>
+			<torque>20</torque>
+			<topicName>cmd_vel</topicName>
+			<broadcastTF>false</broadcastTF>
+		</plugin>
+	</gazebo>
 </robot>

Commit message: Allow passing NS into gazebo plugin

File: sf_robot_description/config/pioneer3dx.xacro (robot description, xacro)
@@ -5,6 +5,8 @@
 	xmlns:interface="http://playerstage.sourceforge.net/gazebo/xmlschema/#interface"
 	xmlns:xacro="http://ros.org/wiki/xacro">
-	<xacro:include filename="$(find sf_robot_description)/config/pioneer3dx_wheel.xacro" />
-	<xacro:include filename="$(find sf_robot_description)/config/pioneer3dx_sonar.xacro" />
+	<xacro:include
+		filename="$(find sf_robot_description)/config/pioneer3dx_wheel.xacro" />
+	<xacro:include
+		filename="$(find sf_robot_description)/config/pioneer3dx_sonar.xacro" />
 	<!-- Chassis -->
 	<link name="base_link">
@@ -74,25 +76,27 @@
 		reflect="1" />
 	<xacro:p3dx_swivel parent="base" />
-	<gazebo>
-		<plugin name="differential_drive_controller" filename="libgazebo_ros_diff_drive.so">
-			<alwaysOn>true</alwaysOn>
-			<rosDebugLevel>na</rosDebugLevel>
-			<updateRate>100.0</updateRate>
-			<robotNamespace>/</robotNamespace>
-			<leftJoint>base_right_wheel_joint</leftJoint>
-			<rightJoint>base_left_wheel_joint</rightJoint>
-			<wheelAcceleration>0</wheelAcceleration>
-			<wheelTorque>200</wheelTorque>
-			<wheelSeparation>0.39</wheelSeparation>
-			<wheelDiameter>0.15</wheelDiameter>
-			<publishTf>false</publishTf>
-			<publishWheelTF>false</publishWheelTF>
-			<publishWheelJointState>false</publishWheelJointState>
-			<commandTopic>cmd_vel</commandTopic>
-			<odometrySource>1</odometrySource>
-			<odometryTopic>odom</odometryTopic>
-			<odometryFrame>odom</odometryFrame>
-			<robotBaseFrame>base_link</robotBaseFrame>
-		</plugin>
-	</gazebo>
+	<xacro:macro name="gazebo_plugin" params="ns">
+		<gazebo>
+			<plugin name="differential_drive_controller" filename="libgazebo_ros_diff_drive.so">
+				<alwaysOn>true</alwaysOn>
+				<rosDebugLevel>na</rosDebugLevel>
+				<updateRate>100.0</updateRate>
+				<robotNamespace>${ns}</robotNamespace>
+				<leftJoint>base_right_wheel_joint</leftJoint>
+				<rightJoint>base_left_wheel_joint</rightJoint>
+				<wheelAcceleration>0</wheelAcceleration>
+				<wheelTorque>200</wheelTorque>
+				<wheelSeparation>0.39</wheelSeparation>
+				<wheelDiameter>0.15</wheelDiameter>
+				<publishTf>true</publishTf>
+				<publishWheelTF>true</publishWheelTF>
+				<publishWheelJointState>true</publishWheelJointState>
+				<commandTopic>cmd_vel</commandTopic>
+				<odometrySource>true</odometrySource>
+				<odometryTopic>odom</odometryTopic>
+				<odometryFrame>odom</odometryFrame>
+				<robotBaseFrame>base_link</robotBaseFrame>
+			</plugin>
+		</gazebo>
+	</xacro:macro>
 </robot>

File: sf_robot_description/config/sf1-1.xacro (robot description, xacro)
@@ -282,13 +282,13 @@
 		</gazebo>
 	</xacro:macro>
-	<xacro:head name="head" parent="head_tilt_hinge">
-		<origin rpy="0 0 0" xyz="0 0 0" />
-	</xacro:head>
-	<xacro:tray name="tray" parent="base">
-		<origin rpy="0 0 0" xyz="0.01 0 0.645" />
-	</xacro:tray>
-	<xacro:neck name="neck" parent="base">
-		<origin rpy="0 0 1.5707" xyz="0 0 0.75" />
-	</xacro:neck>
+<!-- 	<xacro:head name="head" parent="head_tilt_hinge"> -->
+<!-- 		<origin rpy="0 0 0" xyz="0 0 0" /> -->
+<!-- 	</xacro:head> -->
+<!-- 	<xacro:tray name="tray" parent="base"> -->
+<!-- 		<origin rpy="0 0 0" xyz="0.01 0 0.645" /> -->
+<!-- 	</xacro:tray> -->
+<!-- 	<xacro:neck name="neck" parent="base"> -->
+<!-- 		<origin rpy="0 0 1.5707" xyz="0 0 0.75" /> -->
+<!-- 	</xacro:neck> -->
 	<xacro:body name="body" parent="base">
 		<origin rpy="0 0 0" xyz="-0.04 0 0.245" />
@@ -299,4 +299,5 @@
 		<origin rpy="0 0 0" xyz="0.15 0.0 0.245" />
 	</xacro:hokuyo_04lx_laser_ug01>
+	<xacro:gazebo_plugin ns="/sunflower1_1" />
 	<gazebo>
 		<plugin name="gazebo_ros_control" filename="libgazebo_ros_control.so">
