Commit message: Re-enable neck/head joints

File: src/sf_robot_description/robots/sf1-1.xacro (robot description, xacro)
@@ -273,13 +273,13 @@
 		</gazebo>
 	</xacro:macro>
-<!-- 	<xacro:head name="head" parent="head_tilt_hinge"> -->
-<!-- 		<origin rpy="0 0 0" xyz="0 0 0" /> -->
-<!-- 	</xacro:head> -->
-<!-- 	<xacro:tray name="tray" parent="base"> -->
-<!-- 		<origin rpy="0 0 0" xyz="0.01 0 0.645" /> -->
-<!-- 	</xacro:tray> -->
-<!-- 	<xacro:neck name="neck" parent="base"> -->
-<!-- 		<origin rpy="0 0 1.5707" xyz="0 0 0.75" /> -->
-<!-- 	</xacro:neck> -->
+	<xacro:head name="head" parent="head_tilt_hinge">
+		<origin rpy="0 0 0" xyz="0 0 0" />
+	</xacro:head>
+	<xacro:tray name="tray" parent="base">
+		<origin rpy="0 0 0" xyz="0.01 0 0.645" />
+	</xacro:tray>
+	<xacro:neck name="neck" parent="base">
+		<origin rpy="0 0 1.5707" xyz="0 0 0.75" />
+	</xacro:neck>
 	<xacro:body name="body" parent="base">
 		<origin rpy="0 0 0" xyz="-0.04 0 0.245" />
