Commit message: Catkin first pass

File: src/sf_robot_description/robots/pioneer3dx.xacro (robot description, xacro)
@@ -5,6 +5,6 @@
 	xmlns:interface="http://playerstage.sourceforge.net/gazebo/xmlschema/#interface"
 	xmlns:xacro="http://ros.org/wiki/xacro">
-	<xacro:include filename="$(find sf_robot_description)/config/pioneer3dx_wheel.xacro" />
-	<xacro:include filename="$(find sf_robot_description)/config/pioneer3dx_sonar.xacro" />
+	<xacro:include filename="$(find sf_robot_description)/urdf/pioneer3dx/pioneer3dx_wheel.xacro" />
+	<xacro:include filename="$(find sf_robot_description)/urdf/pioneer3dx/pioneer3dx_sonar.xacro" />
 	<!-- Chassis -->
 	<link name="base_link">

File: src/sf_robot_description/robots/sf1-1.xacro (robot description, xacro)
@@ -1,13 +1,13 @@
 <?xml version="1.0"?>
-<robot name="sf11"
+<robot name="sf1_1"
 	xmlns:controller="http://playerstage.sourceforge.net/gazebo/xmlschema/#controller"
 	xmlns:interface="http://playerstage.sourceforge.net/gazebo/xmlschema/#interface"
 	xmlns:sensor="http://playerstage.sourceforge.net/gazebo/xmlschema/#sensor"
 	xmlns:xacro="http://ros.org/wiki/xacro">
-	<xacro:include filename="$(find sf_robot_description)/config/hokuyo_laser.xacro" />
-	<xacro:include filename="$(find sf_dynamixel)/defs/dynamixel_ax12.xacro" />
-	<xacro:include filename="$(find sf_dynamixel)/defs/fp04_02.xacro" />
+	<xacro:include filename="$(find sf_robot_description)/urdf/sensors/hokuyo_laser.xacro" />
+	<xacro:include filename="$(find sf_dynamixel)/urdf/dynamixel_ax12.xacro" />
+	<xacro:include filename="$(find sf_dynamixel)/urdf/fp04_02.xacro" />
+	<xacro:include filename="$(find sf_robot_description)/robots/pioneer3dx.xacro" />
 	<!-- Base -->
-	<xacro:include filename="$(find sf_robot_description)/config/pioneer3dx.xacro" />
 	<joint name="base_plate_joint" type="fixed">
 		<origin rpy="0 0 0" xyz="0 0 0.0085" />
@@ -49,6 +49,5 @@
 			<inertial>
 				<mass value="2" />
-				<inertia ixx="0.001" ixy="0.0" ixz="0.0" iyy="0.001" iyz="0.0"
-					izz="0.001" />
+				<inertia ixx="0.001" ixy="0.0" ixz="0.0" iyy="0.001" iyz="0.0" izz="0.001" />
 			</inertial>
 			<visual>
@@ -83,22 +82,18 @@
 	<!-- Neck -->
 	<xacro:macro name="neck" params="name parent *origin">
-		<xacro:ax12 name="neck_lower" parent="${parent}"
-			minPosition="-1.5707" maxPosition="1.5707" maxVelocity="1">
+		<xacro:ax12 name="neck_lower" parent="${parent}" minPosition="-1.5707" maxPosition="1.5707" maxVelocity="1">
 			<insert_block name="origin" />
 		</xacro:ax12>
 		<xacro:fp04_02 name="neck_lower_hinge" parent="neck_lower">
 		</xacro:fp04_02>
-		<xacro:ax12 name="neck_upper" parent="neck_lower_hinge"
-			minPosition="-1.5707" maxPosition="1.5707" maxVelocity="1">
+		<xacro:ax12 name="neck_upper" parent="neck_lower_hinge" minPosition="-1.5707" maxPosition="1.5707" maxVelocity="1">
 			<origin rpy="0 0 0" xyz="0 0 0" />
 		</xacro:ax12>
 		<xacro:fp04_02 name="neck_upper_hinge" parent="neck_upper">
 		</xacro:fp04_02>
-		<xacro:ax12inverted name="head_pan" parent="neck_upper_hinge"
-			minPosition="-1.5707" maxPosition="1.5707" maxVelocity="1">
+		<xacro:ax12inverted name="head_pan" parent="neck_upper_hinge" minPosition="-1.5707" maxPosition="1.5707" maxVelocity="1">
 			<origin rpy="0 0 -1.57079" xyz="0 0 0" />
 		</xacro:ax12inverted>
-		<xacro:ax12 name="head_tilt" parent="head_pan" minPosition="-1.5707"
-			maxPosition="1.5707" maxVelocity="1">
+		<xacro:ax12 name="head_tilt" parent="head_pan" minPosition="-1.5707" maxPosition="1.5707" maxVelocity="1">
 			<origin rpy="0 0 0" xyz="0 0 0" />
 		</xacro:ax12>
@@ -116,6 +111,5 @@
 			<inertial>
 				<mass value="0.01" />
-				<inertia ixx="0.001" ixy="0.0" ixz="0.0" iyy="0.001" iyz="0.0"
-					izz="0.001" />
+				<inertia ixx="0.001" ixy="0.0" ixz="0.0" iyy="0.001" iyz="0.0" izz="0.001" />
 			</inertial>
 			<visual>
@@ -182,6 +176,5 @@
 			<inertial>
 				<mass value="0.01" />
-				<inertia ixx="0.001" ixy="0.0" ixz="0.0" iyy="0.001" iyz="0.0"
-					izz="0.001" />
+				<inertia ixx="0.001" ixy="0.0" ixz="0.0" iyy="0.001" iyz="0.0" izz="0.001" />
 			</inertial>
 			<visual>
@@ -218,6 +211,5 @@
 			<inertial>
 				<mass value="0.1" />
-				<inertia ixx="0.001" ixy="0.0" ixz="0.0" iyy="0.001" iyz="0.0"
-					izz="0.001" />
+				<inertia ixx="0.001" ixy="0.0" ixz="0.0" iyy="0.001" iyz="0.0" izz="0.001" />
 			</inertial>
 			<visual>
@@ -259,6 +251,5 @@
 				<mass value="10" />
 				<origin xyz="0 0 0.2525" rpy="0 0 0" />
-				<inertia ixx="0.001" ixy="0.0" ixz="0.0" iyy="0.001" iyz="0.0"
-					izz="0.001" />
+				<inertia ixx="0.001" ixy="0.0" ixz="0.0" iyy="0.001" iyz="0.0" izz="0.001" />
 			</inertial>
 			<visual>
@@ -294,7 +285,6 @@
 		<origin rpy="0 0 0" xyz="-0.04 0 0.245" />
 	</xacro:body>
-	<xacro:hokuyo_04lx_laser_ug01 name="base_laser_front"
-		parent="base" ros_topic="scan_front" update_rate="10" min_angle="-2.094"
-		max_angle="2.094">
+	<xacro:hokuyo_04lx_laser_ug01 name="base_laser_front" parent="base" ros_topic="scan_front" update_rate="10"
+		min_angle="-2.094" max_angle="2.094">
 		<origin rpy="0 0 0" xyz="0.15 0.0 0.245" />
 	</xacro:hokuyo_04lx_laser_ug01>

Commit message: more gazebo work

File: src/sf_robot_description/robots/pioneer3dx.xacro (robot description, xacro)
@@ -77,5 +77,5 @@
 		<gazebo>
 			<plugin name="differential_drive_controller" filename="libgazebo_ros_diff_drive.so">
-				<alwaysOn>1</alwaysOn>
+				<alwaysOn>true</alwaysOn>
 				<rosDebugLevel>na</rosDebugLevel>
 				<updateRate>100.0</updateRate>
@@ -84,5 +84,6 @@
 				<rightJoint>base_left_wheel_joint</rightJoint>
 				<wheelAcceleration>0</wheelAcceleration>
-				<wheelTorque>200</wheelTorque>
+				<wheelTorque>5</wheelTorque>
+				<torque>5</torque>
 				<wheelSeparation>0.39</wheelSeparation>
 				<wheelDiameter>0.15</wheelDiameter>

File: src/sf_robot_description/urdf/sensors/hokuyo_laser.xacro (robot description, xacro)
@@ -1,6 +1,5 @@
 <?xml version="1.0"?>
 <robot xmlns:xacro="http://ros.org/wiki/xacro">
-	<xacro:macro name="hokuyo_04lx_laser_ug01"
-		params="name parent *origin ros_topic update_rate min_angle max_angle">
+	<xacro:macro name="hokuyo_04lx_laser_ug01" params="name parent *origin ros_topic update_rate min_angle max_angle">
 		<joint name="${name}_joint" type="fixed">
 			<insert_block name="origin" />
@@ -12,6 +11,5 @@
 				<mass value="0.01" />
 				<origin xyz="0 0 0.0205" rpy="0 0 0" />
-				<inertia ixx="0.001" ixy="0.0" ixz="0.0" iyy="0.001" iyz="0.0"
-					izz="0.001" />
+				<inertia ixx="0.001" ixy="0.0" ixz="0.0" iyy="0.001" iyz="0.0" izz="0.001" />
 			</inertial>
 			<visual>
@@ -43,6 +41,5 @@
 				<mass value="0.01" />
 				<origin xyz="0 0 0.0145" rpy="0 0 0" />
-				<inertia ixx="0.001" ixy="0.0" ixz="0.0" iyy="0.001" iyz="0.0"
-					izz="0.001" />
+				<inertia ixx="0.001" ixy="0.0" ixz="0.0" iyy="0.001" iyz="0.0" izz="0.001" />
 			</inertial>
 			<visual>
@@ -82,4 +79,9 @@
 						<resolution>0.06</resolution>
 					</range>
+					<noise>
+						<type>gaussian</type>
+						<mean>0.0</mean>
+						<stddev>0.01</stddev>
+					</noise>
 				</ray>
 				<plugin name="gazebo_ros_${name}_controller" filename="libgazebo_ros_gpu_laser.so">
