Commit message: Major reorg/simplificatoin of sunflower packages

File: src/dynamixel_description/urdf/dynamixel_ax12.xacro (robot description, xacro)
@@ -9,5 +9,5 @@
 			<visual>
 				<geometry name="ax12mesh">
-					<mesh filename="package://sf_dynamixel/meshes/ax12_box_plain.stl"
+					<mesh filename="package://dynamixel_description/meshes/ax12_box_plain.stl"
 						scale="0.001 0.001 0.001" />
 				</geometry>
@@ -24,5 +24,5 @@
 			<collision>
 				<geometry name="ax12mesh">
-					<mesh filename="package://sf_dynamixel/meshes/ax12_box_plain.stl"
+					<mesh filename="package://dynamixel_description/meshes/ax12_box_plain.stl"
 						scale="0.001 0.001 0.001" />
 				</geometry>
@@ -85,5 +85,5 @@
 			<visual>
 				<geometry name="ax12mesh">
-					<mesh filename="package://sf_dynamixel/meshes/ax12_box_plain.stl"
+					<mesh filename="package://dynamixel_description/meshes/ax12_box_plain.stl"
 						scale="0.001 0.001 0.001" />
 				</geometry>
@@ -100,5 +100,5 @@
 				<origin rpy="1.57075 0 3.14159" xyz="-0.012 0 0.019" />
 				<geometry name="ax12mesh">
-					<mesh filename="package://sf_dynamixel/meshes/ax12_box_plain.stl"
+					<mesh filename="package://dynamixel_description/meshes/ax12_box_plain.stl"
 						scale="0.001 0.001 0.001" />
 				</geometry>

File: src/dynamixel_description/urdf/fp04_02.xacro (robot description, xacro)
@@ -9,5 +9,5 @@
 			<visual>
 				<geometry name="fp04_02mesh">
-					<mesh filename="package://sf_dynamixel/meshes/F2.stl" scale="0.001 0.001 0.001" />
+					<mesh filename="package://dynamixel_description/meshes/F2.stl" scale="0.001 0.001 0.001" />
 				</geometry>
 				<material name="plastic_green">
@@ -18,5 +18,5 @@
 			<collision>
 				<geometry name="fp04_02mesh">
-					<mesh filename="package://sf_dynamixel/meshes/F2.stl" scale="0.001 0.001 0.001" />
+					<mesh filename="package://dynamixel_description/meshes/F2.stl" scale="0.001 0.001 0.001" />
 				</geometry>
 			</collision>

File: src/sf_robot_description/robots/sunflower1_1.xacro (robot description, xacro)
@@ -6,6 +6,6 @@
 	xmlns:xacro="http://ros.org/wiki/xacro">
 	<xacro:include filename="$(find sf_robot_description)/urdf/sensors/hokuyo_laser.xacro" />
-	<xacro:include filename="$(find sf_dynamixel)/urdf/dynamixel_ax12.xacro" />
-	<xacro:include filename="$(find sf_dynamixel)/urdf/fp04_02.xacro" />
+	<xacro:include filename="$(find dynamixel_description)/urdf/dynamixel_ax12.xacro" />
+	<xacro:include filename="$(find dynamixel_description)/urdf/fp04_02.xacro" />
 	<xacro:include filename="$(find sf_robot_description)/robots/pioneer3dx.xacro" />
 	<!-- Base -->

Commit message: Gazebo performance fix: Add simple collision for dynamixel body, disable collision for mounts

File: src/dynamixel_description/urdf/dynamixel_ax12.xacro (robot description, xacro)
@@ -23,7 +23,6 @@
 			</inertial>
 			<collision>
-				<geometry name="ax12mesh">
-					<mesh filename="package://dynamixel_description/meshes/ax12_box_plain.stl"
-						scale="0.001 0.001 0.001" />
+				<geometry name="ax12simple">
+					<box size="0.050 0.038 0.032" />
 				</geometry>
 			</collision>
@@ -44,9 +43,4 @@
 					izz="0.001" />
 			</inertial>
-			<collision>
-				<geometry>
-					<cylinder length="0.005" radius="0.011" />
-				</geometry>
-			</collision>
 		</link>
 		<joint name="${name}_joint" type="revolute">
@@ -99,7 +93,6 @@
 			<collision>
 				<origin rpy="1.57075 0 3.14159" xyz="-0.012 0 0.019" />
-				<geometry name="ax12mesh">
-					<mesh filename="package://dynamixel_description/meshes/ax12_box_plain.stl"
-						scale="0.001 0.001 0.001" />
+				<geometry name="ax12simple">
+					<box size="0.050 0.038 0.032" />
 				</geometry>
 			</collision>

File: src/dynamixel_description/urdf/fp04_02.xacro (robot description, xacro)
@@ -16,9 +16,4 @@
 				<origin rpy="-1.57075 0 1.57075" xyz="0 0 0.0" />
 			</visual>
-			<collision>
-				<geometry name="fp04_02mesh">
-					<mesh filename="package://dynamixel_description/meshes/F2.stl" scale="0.001 0.001 0.001" />
-				</geometry>
-			</collision>
 			<inertial>
 				<mass value="0.005" />

File: src/sf_robot_description/robots/pioneer3dx.xacro (robot description, xacro)
@@ -77,5 +77,5 @@
 		<gazebo>
 			<plugin name="differential_drive_controller" filename="libgazebo_ros_diff_drive.so">
-				<alwaysOn>true</alwaysOn>
+				<alwaysOn>1</alwaysOn>
 				<rosDebugLevel>na</rosDebugLevel>
 				<updateRate>100.0</updateRate>
@@ -87,9 +87,9 @@
 				<wheelSeparation>0.39</wheelSeparation>
 				<wheelDiameter>0.15</wheelDiameter>
-				<publishTf>true</publishTf>
+				<publishTf>1</publishTf>
 				<publishWheelTF>true</publishWheelTF>
 				<publishWheelJointState>true</publishWheelJointState>
 				<commandTopic>cmd_vel</commandTopic>
-				<odometrySource>true</odometrySource>
+				<odometrySource>world</odometrySource>
 				<odometryTopic>odom</odometryTopic>
 				<odometryFrame>odom</odometryFrame>

Commit message: gazebosim work

File: src/dynamixel_description/urdf/dynamixel_ax12.xacro (robot description, xacro)
@@ -1,14 +1,10 @@
 <?xml version="1.0" encoding="UTF-8"?>
-<robot xmlns:controller="http://playerstage.sourceforge.net/gazebo/xmlschema/#controller"
-	xmlns:interface="http://playerstage.sourceforge.net/gazebo/xmlschema/#interface"
-	xmlns:sensor="http://playerstage.sourceforge.net/gazebo/xmlschema/#sensor"
-	xmlns:xacro="http://ros.org/wiki/xacro">
-	<xacro:macro name="ax12"
-		params="name parent minPosition maxPosition maxVelocity *origin">
+<robot xmlns:controller="http://playerstage.sourceforge.net/gazebo/xmlschema/#controller" xmlns:interface="http://playerstage.sourceforge.net/gazebo/xmlschema/#interface"
+	xmlns:sensor="http://playerstage.sourceforge.net/gazebo/xmlschema/#sensor" xmlns:xacro="http://ros.org/wiki/xacro">
+	<xacro:macro name="ax12" params="name parent minPosition maxPosition maxVelocity *origin">
 		<link name="${name}_box_link">
 			<visual>
 				<geometry name="ax12mesh">
-					<mesh filename="package://dynamixel_description/meshes/ax12_box_plain.stl"
-						scale="0.001 0.001 0.001" />
+					<mesh filename="package://dynamixel_description/meshes/ax12_box_plain.stl" scale="0.001 0.001 0.001" />
 				</geometry>
 				<material name="plastic_black">
@@ -19,6 +15,5 @@
 			<inertial>
 				<mass value="0.01" />
-				<inertia ixx="0.001" ixy="0.0" ixz="0.0" iyy="0.001" iyz="0.0"
-					izz="0.001" />
+				<inertia ixx="0.001" ixy="0.0" ixz="0.0" iyy="0.001" iyz="0.0" izz="0.001" />
 			</inertial>
 			<collision>
@@ -40,6 +35,5 @@
 			<inertial>
 				<mass value="0.001" />
-				<inertia ixx="0.001" ixy="0.0" ixz="0.0" iyy="0.001" iyz="0.0"
-					izz="0.001" />
+				<inertia ixx="0.001" ixy="0.0" ixz="0.0" iyy="0.001" iyz="0.0" izz="0.001" />
 			</inertial>
 		</link>
@@ -50,4 +44,5 @@
 			<axis xyz="1 0 0" />
 			<limit effort="0" lower="-1.5707" upper="1.5707" velocity="1" />
+			<dynamics damping="0.1" />
 		</joint>
 		<joint name="${name}_box_joint" type="fixed">
@@ -60,8 +55,8 @@
 			<type>transmission_interface/SimpleTransmission</type>
 			<joint name="${name}_joint">
-				<hardwareInterface>PositionJointInterface</hardwareInterface>
+				<hardwareInterface>EffortJointInterface</hardwareInterface>
 			</joint>
 			<actuator name="${name}_motor">
-				<hardwareInterface>PositionJointInterface</hardwareInterface>
+				<hardwareInterface>EffortJointInterface</hardwareInterface>
 				<mechanicalReduction>1</mechanicalReduction>
 			</actuator>
@@ -74,11 +69,9 @@
 		</gazebo>
 	</xacro:macro>
-	<xacro:macro name="ax12inverted"
-		params="name parent minPosition maxPosition maxVelocity *origin">
+	<xacro:macro name="ax12inverted" params="name parent minPosition maxPosition maxVelocity *origin">
 		<link name="${name}_box_link">
 			<visual>
 				<geometry name="ax12mesh">
-					<mesh filename="package://dynamixel_description/meshes/ax12_box_plain.stl"
-						scale="0.001 0.001 0.001" />
+					<mesh filename="package://dynamixel_description/meshes/ax12_box_plain.stl" scale="0.001 0.001 0.001" />
 				</geometry>
 				<material name="plastic_black" />
@@ -88,6 +81,5 @@
 				<mass value="0.01" />
 				<origin rpy="0 0 0" xyz="-0.012 0 0.019" />
-				<inertia ixx="0.001" ixy="0.0" ixz="0.0" iyy="0.001" iyz="0.0"
-					izz="0.001" />
+				<inertia ixx="0.001" ixy="0.0" ixz="0.0" iyy="0.001" iyz="0.0" izz="0.001" />
 			</inertial>
 			<collision>
@@ -108,6 +100,5 @@
 			<inertial>
 				<mass value="0.001" />
-				<inertia ixx="0.001" ixy="0.0" ixz="0.0" iyy="0.001" iyz="0.0"
-					izz="0.001" />
+				<inertia ixx="0.001" ixy="0.0" ixz="0.0" iyy="0.001" iyz="0.0" izz="0.001" />
 				<origin rpy="0 0 0" xyz="0 0 0.0025" />
 			</inertial>
@@ -141,8 +132,8 @@
 			<type>transmission_interface/SimpleTransmission</type>
 			<joint name="${name}_joint">
-				<hardwareInterface>PositionJointInterface</hardwareInterface>
+				<hardwareInterface>EffortJointInterface</hardwareInterface>
 			</joint>
 			<actuator name="${name}_motor">
-				<hardwareInterface>PositionJointInterface</hardwareInterface>
+				<hardwareInterface>EffortJointInterface</hardwareInterface>
 				<mechanicalReduction>1</mechanicalReduction>
 			</actuator>

File: src/sf_robot_description/robots/pioneer3dx.xacro (robot description, xacro)
@@ -74,5 +74,5 @@
 		reflect="1" />
 	<xacro:p3dx_swivel parent="base" />
-	<xacro:macro name="gazebo_plugin" params="ns">
+	<xacro:macro name="p3dx_gazebo_plugin" params="ns">
 		<gazebo>
 			<plugin name="differential_drive_controller" filename="libgazebo_ros_diff_drive.so">

File: src/sf_robot_description/robots/sunflower1_1.xacro (robot description, xacro)
@@ -1,8 +1,5 @@
 <?xml version="1.0"?>
-<robot name="sf1_1"
-	xmlns:controller="http://playerstage.sourceforge.net/gazebo/xmlschema/#controller"
-	xmlns:interface="http://playerstage.sourceforge.net/gazebo/xmlschema/#interface"
-	xmlns:sensor="http://playerstage.sourceforge.net/gazebo/xmlschema/#sensor"
-	xmlns:xacro="http://ros.org/wiki/xacro">
+<robot name="sf1_1" xmlns:controller="http://playerstage.sourceforge.net/gazebo/xmlschema/#controller" xmlns:interface="http://playerstage.sourceforge.net/gazebo/xmlschema/#interface"
+	xmlns:sensor="http://playerstage.sourceforge.net/gazebo/xmlschema/#sensor" xmlns:xacro="http://ros.org/wiki/xacro">
 	<xacro:include filename="$(find sf_robot_description)/urdf/sensors/hokuyo_laser.xacro" />
 	<xacro:include filename="$(find dynamixel_description)/urdf/dynamixel_ax12.xacro" />
@@ -72,8 +69,8 @@
 			<type>transmission_interface/SimpleTransmission</type>
 			<joint name="${name}_joint">
-				<hardwareInterface>PositionJointInterface</hardwareInterface>
+				<hardwareInterface>EffortJointInterface</hardwareInterface>
 			</joint>
 			<actuator name="${name}_motor">
-				<hardwareInterface>PositionJointInterface</hardwareInterface>
+				<hardwareInterface>EffortJointInterface</hardwareInterface>
 				<mechanicalReduction>1</mechanicalReduction>
 			</actuator>
@@ -415,8 +412,9 @@
 		<origin rpy="0 0 0" xyz="0.15 0.0 0.245" />
 	</xacro:hokuyo_04lx_laser_ug01>
-	<xacro:gazebo_plugin ns="/sunflower1_1" />
+	<xacro:p3dx_gazebo_plugin ns="/sunflower1_1" />
 	<gazebo>
 		<plugin name="gazebo_ros_control" filename="libgazebo_ros_control.so">
 			<robotNamespace>/sunflower1_1</robotNamespace>
+			<robotSimType>gazebo_ros_control/DefaultRobotHWSim</robotSimType>
 		</plugin>
 	</gazebo>
